Commit message: updated coeffs for right forearm

File: common/xacro/serial_numbers/forearm_testbench_serials.xacro (robot description, xacro)
@@ -1,4 +1,4 @@
 <robot xmlns:xacro="http://ros.org/wiki/xacro" name="forearm_testbench">
-	<xacro:property name="testbench_serial_number" value="v_g_005" />
-	<xacro:property name="forearm_serial_number" value="v_h_001" />
+	<xacro:property name="testbench_serial_number" value="v_g_003" />
+	<xacro:property name="forearm_serial_number" value="v_h_002" />
 </robot>
