Commit message: swapped left and right leg serials for val D

File: common/xacro/serial_numbers/valkyrie_D_serials.xacro (robot description, xacro)
@@ -1,3 +1,4 @@
 <robot xmlns:xacro="http://ros.org/wiki/xacro" name="valkyrie_D_serials">
+    <!--  Original
     <xacro:property name="leftLegJ1SerialNumber" value="v_a_017" />
     <xacro:property name="leftLegJ2SerialNumber" value="v_b_011" />
@@ -5,5 +6,12 @@
     <xacro:property name="leftLegJ4SerialNumber" value="v_d_007" />
     <xacro:property name="leftAnkleLeftActuatorSerialNumber" value="v_e_009" />
-    <xacro:property name="leftAnkleRightActuatorSerialNumber" value="v_e_010" />
+    <xacro:property name="leftAnkleRightActuatorSerialNumber" value="v_e_010" /> -->
+    <xacro:property name="rightLegJ1SerialNumber" value="v_a_017" />
+    <xacro:property name="rightLegJ2SerialNumber" value="v_b_011" />
+    <xacro:property name="rightLegJ3SerialNumber" value="v_c_007" />
+    <xacro:property name="rightLegJ4SerialNumber" value="v_d_007" />
+    <xacro:property name="rightAnkleLeftActuatorSerialNumber" value="v_e_009" />
+    <xacro:property name="rightAnkleRightActuatorSerialNumber" value="v_e_010" />
+    <!--  Original
     <xacro:property name="rightLegJ1SerialNumber" value="v_a_018" />
     <xacro:property name="rightLegJ2SerialNumber" value="v_b_010" />
@@ -11,5 +19,11 @@
     <xacro:property name="rightLegJ4SerialNumber" value="v_d_006" />
     <xacro:property name="rightAnkleRightActuatorSerialNumber" value="v_e_008" />
-    <xacro:property name="rightAnkleLeftActuatorSerialNumber" value="v_e_007" />
+    <xacro:property name="rightAnkleLeftActuatorSerialNumber" value="v_e_007" /> -->
+    <xacro:property name="leftLegJ1SerialNumber" value="v_a_018" />
+    <xacro:property name="leftLegJ2SerialNumber" value="v_b_010" />
+    <xacro:property name="leftLegJ3SerialNumber" value="v_c_006" />
+    <xacro:property name="leftLegJ4SerialNumber" value="v_d_006" />
+    <xacro:property name="leftAnkleRightActuatorSerialNumber" value="v_e_008" />
+    <xacro:property name="leftAnkleLeftActuatorSerialNumber" value="v_e_007" />
     <xacro:property name="leftArmJ1SerialNumber" value="v_a_019" />
     <xacro:property name="leftArmJ2SerialNumber" value="v_b_014" />
