Commit message: starting to update to use new package and config file for sensors

File: common/xacro/serial_numbers/valkyrie_A_serials.xacro (robot description, xacro)
@@ -33,3 +33,6 @@
 	<xacro:property name="right_foot_ATI_serial" value="FT16592" />
 	<xacro:property name="sim_ATI_serial" value="FT001SIM" />
+	<xacro:property name="pelvis_middle_imu_serial" value="000001" />
+	<xacro:property name="pelvis_rear_imu_serial" value="47095" />
+	<xacro:property name="torso_left_imu_serial" value="47090" />
 </robot>

File: common/xacro/serial_numbers/valkyrie_B_serials.xacro (robot description, xacro)
@@ -33,3 +33,6 @@
 	<xacro:property name="right_foot_ATI_serial" value="FT14018" />
     <xacro:property name="sim_ATI_serial" value="FT001SIM" />
+    <xacro:property name="pelvis_middle_imu_serial" value="000001" />
+	<xacro:property name="pelvis_rear_imu_serial" value="47095" />
+	<xacro:property name="torso_left_imu_serial" value="47090" />
 </robot>

File: common/xacro/serial_numbers/valkyrie_C_serials.xacro (robot description, xacro)
@@ -33,3 +33,6 @@
 	<xacro:property name="right_foot_ATI_serial" value="FT17214" />
 	<xacro:property name="sim_ATI_serial" value="FT001SIM" />
+	<xacro:property name="pelvis_middle_imu_serial" value="000001" />
+	<xacro:property name="pelvis_rear_imu_serial" value="47095" />
+	<xacro:property name="torso_left_imu_serial" value="47090" />
 </robot>

File: common/xacro/serial_numbers/valkyrie_D_serials.xacro (robot description, xacro)
@@ -33,3 +33,6 @@
     <xacro:property name="right_foot_ATI_serial" value="FT16590" />
     <xacro:property name="sim_ATI_serial" value="FT001SIM" />
+    <xacro:property name="pelvis_middle_imu_serial" value="000001" />
+    <xacro:property name="pelvis_rear_imu_serial" value="47095" />
+    <xacro:property name="torso_left_imu_serial" value="47090" />
 </robot>

File: model/robots/valkyrie_A.xacro (robot description, xacro)
@@ -6,4 +6,5 @@
     <xacro:include filename="$(find val_description)/common/xacro/serial_numbers/valkyrie_A_serials.xacro"/>
     <xacro:include filename="$(find val_description)/common/xacro/api/valkyrie_A_api.xacro"/>
+    <xacro:include filename="$(find val_description)/common/xacro/config_packages/valkyrie_A_pkg.xacro"/>
     <xacro:include filename="$(find val_description)/common/xacro/dev_ports/valkyrie_A_ports.xacro"/>
 </robot>

File: model/robots/valkyrie_A_arm_mass_sims.xacro (robot description, xacro)
@@ -6,4 +6,5 @@
     <xacro:include filename="$(find val_description)/common/xacro/serial_numbers/valkyrie_A_serials.xacro"/>
     <xacro:include filename="$(find val_description)/common/xacro/api/valkyrie_A_api.xacro"/>
+    <xacro:include filename="$(find val_description)/common/xacro/config_packages/valkyrie_A_pkg.xacro"/>
     <xacro:include filename="$(find val_description)/common/xacro/dev_ports/valkyrie_A_ports.xacro"/>
 </robot>

File: model/robots/valkyrie_B.xacro (robot description, xacro)
@@ -6,4 +6,5 @@
     <xacro:include filename="$(find val_description)/common/xacro/serial_numbers/valkyrie_B_serials.xacro"/>
     <xacro:include filename="$(find val_description)/common/xacro/api/valkyrie_B_api.xacro"/>
+    <xacro:include filename="$(find val_description)/common/xacro/config_packages/valkyrie_B_pkg.xacro"/>
     <xacro:include filename="$(find val_description)/common/xacro/dev_ports/valkyrie_B_ports.xacro"/>
 </robot>

File: model/robots/valkyrie_B_arm_mass_sims.xacro (robot description, xacro)
@@ -6,4 +6,5 @@
     <xacro:include filename="$(find val_description)/common/xacro/serial_numbers/valkyrie_B_serials.xacro"/>
     <xacro:include filename="$(find val_description)/common/xacro/api/valkyrie_B_api.xacro"/>
+    <xacro:include filename="$(find val_description)/common/xacro/config_packages/valkyrie_B_pkg.xacro"/>
     <xacro:include filename="$(find val_description)/common/xacro/dev_ports/valkyrie_B_ports.xacro"/>
 </robot>

File: model/robots/valkyrie_C.xacro (robot description, xacro)
@@ -6,4 +6,5 @@
     <xacro:include filename="$(find val_description)/common/xacro/serial_numbers/valkyrie_C_serials.xacro"/>
     <xacro:include filename="$(find val_description)/common/xacro/api/valkyrie_C_api.xacro"/>
+    <xacro:include filename="$(find val_description)/common/xacro/config_packages/valkyrie_C_pkg.xacro"/>
     <xacro:include filename="$(find val_description)/common/xacro/dev_ports/valkyrie_C_ports.xacro"/>
 </robot>

File: model/robots/valkyrie_C_arm_mass_sims.xacro (robot description, xacro)
@@ -6,4 +6,5 @@
     <xacro:include filename="$(find val_description)/common/xacro/serial_numbers/valkyrie_C_serials.xacro"/>
     <xacro:include filename="$(find val_description)/common/xacro/api/valkyrie_C_api.xacro"/>
+    <xacro:include filename="$(find val_description)/common/xacro/config_packages/valkyrie_C_pkg.xacro"/>
     <xacro:include filename="$(find val_description)/common/xacro/dev_ports/valkyrie_C_ports.xacro"/>
 </robot>

File: model/robots/valkyrie_D.xacro (robot description, xacro)
@@ -6,4 +6,5 @@
     <xacro:include filename="$(find val_description)/common/xacro/serial_numbers/valkyrie_D_serials.xacro"/>
     <xacro:include filename="$(find val_description)/common/xacro/api/valkyrie_D_api.xacro"/>
+    <xacro:include filename="$(find val_description)/common/xacro/config_packages/valkyrie_D_pkg.xacro"/>
     <xacro:include filename="$(find val_description)/common/xacro/dev_ports/valkyrie_D_ports.xacro"/>
 </robot>

File: model/robots/valkyrie_D_arm_mass_sims.xacro (robot description, xacro)
@@ -6,4 +6,5 @@
     <xacro:include filename="$(find val_description)/common/xacro/serial_numbers/valkyrie_D_serials.xacro"/>
     <xacro:include filename="$(find val_description)/common/xacro/api/valkyrie_D_api.xacro"/>
+    <xacro:include filename="$(find val_description)/common/xacro/config_packages/valkyrie_D_pkg.xacro"/>
     <xacro:include filename="$(find val_description)/common/xacro/dev_ports/valkyrie_D_ports.xacro"/>
 </robot>

File: model/robots/valkyrie_sim.xacro (robot description, xacro)
@@ -11,4 +11,5 @@
     <xacro:include filename="$(find val_description)/model/urdf/multisense_sl.urdf" />
     <xacro:include filename="$(find val_description)/common/xacro/serial_numbers/valkyrie_A_serials.xacro"/>
+    <xacro:include filename="$(find val_description)/common/xacro/config_packages/valkyrie_A_pkg.xacro"/>
     <xacro:include filename="$(find val_description)/common/xacro/dev_ports/valkyrie_gazebo_ports.xacro"/>
     <xacro:include filename="$(find val_description)/model/robots/common/xacro/valkyrie_base_sim.xacro"/>

File: model/robots/valkyrie_sim_arm_mass_sims.xacro (robot description, xacro)
@@ -11,4 +11,5 @@
     <xacro:include filename="$(find val_description)/model/urdf/multisense_sl.urdf" />
     <xacro:include filename="$(find val_description)/common/xacro/serial_numbers/valkyrie_A_serials.xacro"/>
+    <xacro:include filename="$(find val_description)/common/xacro/config_packages/valkyrie_A_pkg.xacro"/>
     <xacro:include filename="$(find val_description)/common/xacro/dev_ports/valkyrie_gazebo_ports.xacro"/>
     <xacro:include filename="$(find val_description)/model/robots/common/xacro/valkyrie_arm_mass_sims_base_sim.xacro"/>

File: model/robots/valkyrie_sim_gazebo_sync.xacro (robot description, xacro)
@@ -12,4 +12,5 @@
     <xacro:include filename="$(find val_description)/model/urdf/multisense_sl.urdf" />
     <xacro:include filename="$(find val_description)/common/xacro/serial_numbers/valkyrie_A_serials.xacro"/>
+    <xacro:include filename="$(find val_description)/common/xacro/config_packages/valkyrie_A_pkg.xacro"/>
     <xacro:include filename="$(find val_description)/common/xacro/dev_ports/valkyrie_gazebo_ports.xacro"/>
     <xacro:include filename="$(find val_description)/model/robots/common/xacro/valkyrie_base_sim.xacro"/>

Commit message: Serial swap.

File: common/xacro/serial_numbers/valkyrie_A_serials.xacro (robot description, xacro)
@@ -7,9 +7,9 @@
 	<xacro:property name="leftAnkleRightActuatorSerialNumber" value="v_e_015" />
 	<xacro:property name="rightLegJ1SerialNumber" value="v_a_003" />
-	<xacro:property name="rightLegJ2SerialNumber" value="v_b_001" />
-	<xacro:property name="rightLegJ3SerialNumber" value="v_c_001" />
-	<xacro:property name="rightLegJ4SerialNumber" value="v_d_004" />
-	<xacro:property name="rightAnkleLeftActuatorSerialNumber" value="v_e_003" />
-	<xacro:property name="rightAnkleRightActuatorSerialNumber" value="v_e_004" />
+	<xacro:property name="rightLegJ2SerialNumber" value="v_b_015" />
+    <xacro:property name="rightLegJ3SerialNumber" value="v_c_009" />
+    <xacro:property name="rightLegJ4SerialNumber" value="v_d_009" />
+    <xacro:property name="rightAnkleLeftActuatorSerialNumber" value="v_e_021" />
+    <xacro:property name="rightAnkleRightActuatorSerialNumber" value="v_e_022" />
 	<xacro:property name="leftArmJ1SerialNumber" value="v_a_005" />
 	<xacro:property name="leftArmJ2SerialNumber" value="v_b_004" />
@@ -31,5 +31,5 @@
     <xacro:property name="rightForearmSerialNumber" value="v_h_008"/>
 	<xacro:property name="left_foot_ATI_serial" value="FT17218" />
-	<xacro:property name="right_foot_ATI_serial" value="FT16592" />
+	<xacro:property name="right_foot_ATI_serial" value="FT14018" />
 	<xacro:property name="sim_ATI_serial" value="FT001SIM" />
 </robot>

File: common/xacro/serial_numbers/valkyrie_B_serials.xacro (robot description, xacro)
@@ -7,9 +7,9 @@
     <xacro:property name="leftAnkleRightActuatorSerialNumber" value="v_e_020" />
 	<xacro:property name="rightLegJ1SerialNumber" value="v_a_007" />
-	<xacro:property name="rightLegJ2SerialNumber" value="v_b_015" />
-    <xacro:property name="rightLegJ3SerialNumber" value="v_c_009" />
-    <xacro:property name="rightLegJ4SerialNumber" value="v_d_009" />
-    <xacro:property name="rightAnkleLeftActuatorSerialNumber" value="v_e_021" />
-    <xacro:property name="rightAnkleRightActuatorSerialNumber" value="v_e_022" />
+	<xacro:property name="rightLegJ2SerialNumber" value="v_b_001" />
+	<xacro:property name="rightLegJ3SerialNumber" value="v_c_001" />
+	<xacro:property name="rightLegJ4SerialNumber" value="v_d_004" />
+	<xacro:property name="rightAnkleLeftActuatorSerialNumber" value="v_e_003" />
+	<xacro:property name="rightAnkleRightActuatorSerialNumber" value="v_e_004" />
 	<xacro:property name="leftArmJ1SerialNumber" value="v_a_002" />
 	<xacro:property name="leftArmJ2SerialNumber" value="v_b_005" />
@@ -31,5 +31,5 @@
     <xacro:property name="rightForearmSerialNumber" value="v_h_004"/>
 	<xacro:property name="left_foot_ATI_serial" value="FT16594" />
-	<xacro:property name="right_foot_ATI_serial" value="FT14018" />
+	<xacro:property name="right_foot_ATI_serial" value="FT16592" />
     <xacro:property name="sim_ATI_serial" value="FT001SIM" />
 </robot>

Commit message: updating serials for mit right leg test

File: common/xacro/serial_numbers/valkyrie_A_serials.xacro (robot description, xacro)
@@ -1,15 +1,15 @@
 <robot xmlns:xacro="http://ros.org/wiki/xacro" name="valkyrie_A_serials">
 	<xacro:property name="leftLegJ1SerialNumber" value="v_a_006" />
-	<xacro:property name="leftLegJ2SerialNumber" value="v_b_006" />
-    <xacro:property name="leftLegJ3SerialNumber" value="v_c_004" />
-    <xacro:property name="leftLegJ4SerialNumber" value="v_d_003" />
-    <xacro:property name="leftAnkleLeftActuatorSerialNumber" value="v_e_016" />
-	<xacro:property name="leftAnkleRightActuatorSerialNumber" value="v_e_015" />
-	<xacro:property name="rightLegJ1SerialNumber" value="v_a_003" />
-	<xacro:property name="rightLegJ2SerialNumber" value="v_b_015" />
-    <xacro:property name="rightLegJ3SerialNumber" value="v_c_009" />
-    <xacro:property name="rightLegJ4SerialNumber" value="v_d_009" />
-    <xacro:property name="rightAnkleLeftActuatorSerialNumber" value="v_e_021" />
-    <xacro:property name="rightAnkleRightActuatorSerialNumber" value="v_e_022" />
+	<xacro:property name="leftLegJ2SerialNumber" value="v_b_016" />
+        <xacro:property name="leftLegJ3SerialNumber" value="v_c_008" />
+        <xacro:property name="leftLegJ4SerialNumber" value="v_d_008" />
+        <xacro:property name="leftAnkleLeftActuatorSerialNumber" value="v_e_019" />
+   	<xacro:property name="leftAnkleRightActuatorSerialNumber" value="v_e_020" />
+	 <xacro:property name="rightLegJ1SerialNumber" value="v_a_003" />
+        <xacro:property name="rightLegJ2SerialNumber" value="v_b_001" />
+        <xacro:property name="rightLegJ3SerialNumber" value="v_c_001" />
+        <xacro:property name="rightLegJ4SerialNumber" value="v_d_004" />
+        <xacro:property name="rightAnkleLeftActuatorSerialNumber" value="v_e_003" />
+        <xacro:property name="rightAnkleRightActuatorSerialNumber" value="v_e_004" />
 	<xacro:property name="leftArmJ1SerialNumber" value="v_a_005" />
 	<xacro:property name="leftArmJ2SerialNumber" value="v_b_004" />

File: common/xacro/serial_numbers/valkyrie_B_serials.xacro (robot description, xacro)
@@ -1,15 +1,15 @@
 <robot xmlns:xacro="http://ros.org/wiki/xacro" name="valkyrie_B_serials">
 	<xacro:property name="leftLegJ1SerialNumber" value="v_a_009" />
-    <xacro:property name="leftLegJ2SerialNumber" value="v_b_016" />
-	<xacro:property name="leftLegJ3SerialNumber" value="v_c_008" />
-	<xacro:property name="leftLegJ4SerialNumber" value="v_d_008" />
-	<xacro:property name="leftAnkleLeftActuatorSerialNumber" value="v_e_019" />
-    <xacro:property name="leftAnkleRightActuatorSerialNumber" value="v_e_020" />
+    <xacro:property name="leftLegJ2SerialNumber" value="v_b_006" />
+	<xacro:property name="leftLegJ3SerialNumber" value="v_c_004" />
+	<xacro:property name="leftLegJ4SerialNumber" value="v_d_003" />
+	<xacro:property name="leftAnkleLeftActuatorSerialNumber" value="v_e_015" />
+    <xacro:property name="leftAnkleRightActuatorSerialNumber" value="v_e_016" />
 	<xacro:property name="rightLegJ1SerialNumber" value="v_a_007" />
-	<xacro:property name="rightLegJ2SerialNumber" value="v_b_001" />
-	<xacro:property name="rightLegJ3SerialNumber" value="v_c_001" />
-	<xacro:property name="rightLegJ4SerialNumber" value="v_d_004" />
-	<xacro:property name="rightAnkleLeftActuatorSerialNumber" value="v_e_003" />
-	<xacro:property name="rightAnkleRightActuatorSerialNumber" value="v_e_004" />
+	<xacro:property name="rightLegJ2SerialNumber" value="v_b_015" />
+	<xacro:property name="rightLegJ3SerialNumber" value="v_c_009" />
+	<xacro:property name="rightLegJ4SerialNumber" value="v_d_009" />
+	<xacro:property name="rightAnkleLeftActuatorSerialNumber" value="v_e_022" />
+	<xacro:property name="rightAnkleRightActuatorSerialNumber" value="v_e_0021" />
 	<xacro:property name="leftArmJ1SerialNumber" value="v_a_002" />
 	<xacro:property name="leftArmJ2SerialNumber" value="v_b_005" />

Commit message: Fixed some indents.

File: common/xacro/serial_numbers/valkyrie_A_serials.xacro (robot description, xacro)
@@ -2,14 +2,14 @@
 	<xacro:property name="leftLegJ1SerialNumber" value="v_a_006" />
 	<xacro:property name="leftLegJ2SerialNumber" value="v_b_016" />
-        <xacro:property name="leftLegJ3SerialNumber" value="v_c_008" />
-        <xacro:property name="leftLegJ4SerialNumber" value="v_d_008" />
-        <xacro:property name="leftAnkleLeftActuatorSerialNumber" value="v_e_019" />
+    <xacro:property name="leftLegJ3SerialNumber" value="v_c_008" />
+    <xacro:property name="leftLegJ4SerialNumber" value="v_d_008" />
+    <xacro:property name="leftAnkleLeftActuatorSerialNumber" value="v_e_019" />
    	<xacro:property name="leftAnkleRightActuatorSerialNumber" value="v_e_020" />
 	 <xacro:property name="rightLegJ1SerialNumber" value="v_a_003" />
-        <xacro:property name="rightLegJ2SerialNumber" value="v_b_001" />
-        <xacro:property name="rightLegJ3SerialNumber" value="v_c_001" />
-        <xacro:property name="rightLegJ4SerialNumber" value="v_d_004" />
-        <xacro:property name="rightAnkleLeftActuatorSerialNumber" value="v_e_003" />
-        <xacro:property name="rightAnkleRightActuatorSerialNumber" value="v_e_004" />
+    <xacro:property name="rightLegJ2SerialNumber" value="v_b_001" />
+    <xacro:property name="rightLegJ3SerialNumber" value="v_c_001" />
+    <xacro:property name="rightLegJ4SerialNumber" value="v_d_004" />
+    <xacro:property name="rightAnkleLeftActuatorSerialNumber" value="v_e_003" />
+    <xacro:property name="rightAnkleRightActuatorSerialNumber" value="v_e_004" />
 	<xacro:property name="leftArmJ1SerialNumber" value="v_a_005" />
 	<xacro:property name="leftArmJ2SerialNumber" value="v_b_004" />

Commit message: calibrated A with MIT left leg

File: common/xacro/serial_numbers/valkyrie_A_serials.xacro (robot description, xacro)
@@ -30,5 +30,5 @@
 	<xacro:property name="leftForearmSerialNumber" value="v_h_007"/>
     <xacro:property name="rightForearmSerialNumber" value="v_h_008"/>
-	<xacro:property name="left_foot_ATI_serial" value="FT17218" />
+	<xacro:property name="left_foot_ATI_serial" value="FT16594" />
 	<xacro:property name="right_foot_ATI_serial" value="FT14018" />
 	<xacro:property name="sim_ATI_serial" value="FT001SIM" />

File: common/xacro/serial_numbers/valkyrie_B_serials.xacro (robot description, xacro)
@@ -30,5 +30,5 @@
 	<xacro:property name="leftForearmSerialNumber" value="v_h_003"/>
     <xacro:property name="rightForearmSerialNumber" value="v_h_004"/>
-	<xacro:property name="left_foot_ATI_serial" value="FT16594" />
+	<xacro:property name="left_foot_ATI_serial" value="FT17218" />
 	<xacro:property name="right_foot_ATI_serial" value="FT16592" />
     <xacro:property name="sim_ATI_serial" value="FT001SIM" />

Commit message: WACKY COEFFS HERE. FIX BEFORE PUSHING TO DEVELOP.

File: common/xacro/serial_numbers/valkyrie_A_serials.xacro (robot description, xacro)
@@ -2,14 +2,14 @@
 	<xacro:property name="leftLegJ1SerialNumber" value="v_a_006" />
 	<xacro:property name="leftLegJ2SerialNumber" value="v_b_016" />
-    <xacro:property name="leftLegJ3SerialNumber" value="v_c_008" />
-    <xacro:property name="leftLegJ4SerialNumber" value="v_d_008" />
-    <xacro:property name="leftAnkleLeftActuatorSerialNumber" value="v_e_019" />
-   	<xacro:property name="leftAnkleRightActuatorSerialNumber" value="v_e_020" />
+    	<xacro:property name="leftLegJ3SerialNumber" value="v_c_008" />
+    	<xacro:property name="leftLegJ4SerialNumber" value="v_d_008" />
+	<xacro:property name="leftAnkleLeftActuatorSerialNumber" value="v_e_016" />
+   	<xacro:property name="leftAnkleRightActuatorSerialNumber" value="v_e_015" />
 	 <xacro:property name="rightLegJ1SerialNumber" value="v_a_003" />
-    <xacro:property name="rightLegJ2SerialNumber" value="v_b_001" />
-    <xacro:property name="rightLegJ3SerialNumber" value="v_c_001" />
-    <xacro:property name="rightLegJ4SerialNumber" value="v_d_004" />
-    <xacro:property name="rightAnkleLeftActuatorSerialNumber" value="v_e_003" />
-    <xacro:property name="rightAnkleRightActuatorSerialNumber" value="v_e_004" />
+	<xacro:property name="rightLegJ2SerialNumber" value="v_b_015" />
+        <xacro:property name="rightLegJ3SerialNumber" value="v_c_009" />
+        <xacro:property name="rightLegJ4SerialNumber" value="v_d_009" />
+        <xacro:property name="rightAnkleLeftActuatorSerialNumber" value="v_e_021" />
+        <xacro:property name="rightAnkleRightActuatorSerialNumber" value="v_e_022" />
 	<xacro:property name="leftArmJ1SerialNumber" value="v_a_005" />
 	<xacro:property name="leftArmJ2SerialNumber" value="v_b_004" />
@@ -30,6 +30,6 @@
 	<xacro:property name="leftForearmSerialNumber" value="v_h_007"/>
     <xacro:property name="rightForearmSerialNumber" value="v_h_008"/>
-	<xacro:property name="left_foot_ATI_serial" value="FT16594" />
-	<xacro:property name="right_foot_ATI_serial" value="FT14018" />
+	<xacro:property name="left_foot_ATI_serial" value="FT17218" />
+	<xacro:property name="right_foot_ATI_serial" value="FT16592" />
 	<xacro:property name="sim_ATI_serial" value="FT001SIM" />
 </robot>

File: common/xacro/serial_numbers/valkyrie_B_serials.xacro (robot description, xacro)
@@ -1,15 +1,15 @@
 <robot xmlns:xacro="http://ros.org/wiki/xacro" name="valkyrie_B_serials">
 	<xacro:property name="leftLegJ1SerialNumber" value="v_a_009" />
-    <xacro:property name="leftLegJ2SerialNumber" value="v_b_006" />
+	<xacro:property name="leftLegJ2SerialNumber" value="v_b_006" />
 	<xacro:property name="leftLegJ3SerialNumber" value="v_c_004" />
 	<xacro:property name="leftLegJ4SerialNumber" value="v_d_003" />
-	<xacro:property name="leftAnkleLeftActuatorSerialNumber" value="v_e_015" />
-    <xacro:property name="leftAnkleRightActuatorSerialNumber" value="v_e_016" />
+    <xacro:property name="leftAnkleLeftActuatorSerialNumber" value="v_e_019" />
+   	<xacro:property name="leftAnkleRightActuatorSerialNumber" value="v_e_020" />
 	<xacro:property name="rightLegJ1SerialNumber" value="v_a_007" />
-	<xacro:property name="rightLegJ2SerialNumber" value="v_b_015" />
-	<xacro:property name="rightLegJ3SerialNumber" value="v_c_009" />
-	<xacro:property name="rightLegJ4SerialNumber" value="v_d_009" />
-	<xacro:property name="rightAnkleLeftActuatorSerialNumber" value="v_e_022" />
-	<xacro:property name="rightAnkleRightActuatorSerialNumber" value="v_e_0021" />
+	<xacro:property name="rightLegJ2SerialNumber" value="v_b_001" />
+    	<xacro:property name="rightLegJ3SerialNumber" value="v_c_001" />
+   	<xacro:property name="rightLegJ4SerialNumber" value="v_d_004" />
+    	<xacro:property name="rightAnkleLeftActuatorSerialNumber" value="v_e_003" />
+    	<xacro:property name="rightAnkleRightActuatorSerialNumber" value="v_e_004" />
 	<xacro:property name="leftArmJ1SerialNumber" value="v_a_002" />
 	<xacro:property name="leftArmJ2SerialNumber" value="v_b_005" />
@@ -30,6 +30,6 @@
 	<xacro:property name="leftForearmSerialNumber" value="v_h_003"/>
     <xacro:property name="rightForearmSerialNumber" value="v_h_004"/>
-	<xacro:property name="left_foot_ATI_serial" value="FT17218" />
-	<xacro:property name="right_foot_ATI_serial" value="FT16592" />
+	<xacro:property name="left_foot_ATI_serial" value="FT16594" />
+	<xacro:property name="right_foot_ATI_serial" value="FT14018" />
     <xacro:property name="sim_ATI_serial" value="FT001SIM" />
 </robot>

Commit message: updating serials temp

File: common/xacro/serial_numbers/valkyrie_A_serials.xacro (robot description, xacro)
@@ -21,5 +21,5 @@
 	<xacro:property name="rightArmJ3SerialNumber" value="v_f_004" />
 	<xacro:property name="rightArmJ4SerialNumber" value="v_f_003" />
-	<xacro:property name="rightArmJ5SerialNumber" value="v_g_017" />
+	<xacro:property name="rightArmJ5SerialNumber" value="v_g_003" />
 	<xacro:property name="neckJ1SerialNumber" value="v_g_006" />
 	<xacro:property name="neckJ2SerialNumber" value="v_g_007" />
@@ -29,5 +29,5 @@
 	<xacro:property name="waistLeftActuatorSerialNumber" value="v_e_006" />
 	<xacro:property name="leftForearmSerialNumber" value="v_h_001"/>
-    	<xacro:property name="rightForearmSerialNumber" value="v_h_008"/>
+    	<xacro:property name="rightForearmSerialNumber" value="v_h_002"/>
 	<xacro:property name="left_foot_ATI_serial" value="FT17218" />
 	<xacro:property name="right_foot_ATI_serial" value="FT14018" />
