Commit message: swaping unit A and unit D leg serials

File: common/xacro/serial_numbers/valkyrie_A_serials.xacro (robot description, xacro)
@@ -1,15 +1,15 @@
 <robot xmlns:xacro="http://ros.org/wiki/xacro" name="valkyrie_A_serials">
 	<xacro:property name="leftLegJ1SerialNumber" value="v_a_006" />
-    <xacro:property name="leftLegJ2SerialNumber" value="v_b_011" />
-    <xacro:property name="leftLegJ3SerialNumber" value="v_c_007" />
-    <xacro:property name="leftLegJ4SerialNumber" value="v_d_007" />
-    <xacro:property name="leftAnkleLeftActuatorSerialNumber" value="v_e_009" />
-    <xacro:property name="leftAnkleRightActuatorSerialNumber" value="v_e_010" />
+       <xacro:property name="leftLegJ2SerialNumber" value="v_b_016" />
+    <xacro:property name="leftLegJ3SerialNumber" value="v_c_008" />
+    <xacro:property name="leftLegJ4SerialNumber" value="v_d_008" />
+    <xacro:property name="leftAnkleLeftActuatorSerialNumber" value="v_e_016" />
+        <xacro:property name="leftAnkleRightActuatorSerialNumber" value="v_e_015" />
 	<xacro:property name="rightLegJ1SerialNumber" value="v_a_003" />
-    <xacro:property name="rightLegJ2SerialNumber" value="v_b_010" />
-    <xacro:property name="rightLegJ3SerialNumber" value="v_c_006" />
-    <xacro:property name="rightLegJ4SerialNumber" value="v_d_006" />
-    <xacro:property name="rightAnkleRightActuatorSerialNumber" value="v_e_008" />
-    <xacro:property name="rightAnkleLeftActuatorSerialNumber" value="v_e_007" />
+        <xacro:property name="rightLegJ2SerialNumber" value="v_b_015" />
+        <xacro:property name="rightLegJ3SerialNumber" value="v_c_009" />
+        <xacro:property name="rightLegJ4SerialNumber" value="v_d_009" />
+        <xacro:property name="rightAnkleLeftActuatorSerialNumber" value="v_e_021" />
+        <xacro:property name="rightAnkleRightActuatorSerialNumber" value="v_e_022" />
 	<xacro:property name="leftArmJ1SerialNumber" value="v_a_005" />
 	<xacro:property name="leftArmJ2SerialNumber" value="v_b_004" />

File: common/xacro/serial_numbers/valkyrie_D_serials.xacro (robot description, xacro)
@@ -1,15 +1,15 @@
 <robot xmlns:xacro="http://ros.org/wiki/xacro" name="valkyrie_D_serials">
     <xacro:property name="leftLegJ1SerialNumber" value="v_a_017" />
-	<xacro:property name="leftLegJ2SerialNumber" value="v_b_016" />
-    <xacro:property name="leftLegJ3SerialNumber" value="v_c_008" />
-    <xacro:property name="leftLegJ4SerialNumber" value="v_d_008" />
-    <xacro:property name="leftAnkleLeftActuatorSerialNumber" value="v_e_016" />
-	<xacro:property name="leftAnkleRightActuatorSerialNumber" value="v_e_015" />
+    <xacro:property name="leftLegJ2SerialNumber" value="v_b_011" />
+    <xacro:property name="leftLegJ3SerialNumber" value="v_c_007" />
+    <xacro:property name="leftLegJ4SerialNumber" value="v_d_007" />
+    <xacro:property name="leftAnkleLeftActuatorSerialNumber" value="v_e_009" />
+    <xacro:property name="leftAnkleRightActuatorSerialNumber" value="v_e_010" />
     <xacro:property name="rightLegJ1SerialNumber" value="v_a_018" />
-	<xacro:property name="rightLegJ2SerialNumber" value="v_b_015" />
-	<xacro:property name="rightLegJ3SerialNumber" value="v_c_009" />
-	<xacro:property name="rightLegJ4SerialNumber" value="v_d_009" />
-	<xacro:property name="rightAnkleLeftActuatorSerialNumber" value="v_e_021" />
-	<xacro:property name="rightAnkleRightActuatorSerialNumber" value="v_e_022" />
+    <xacro:property name="rightLegJ2SerialNumber" value="v_b_010" />
+    <xacro:property name="rightLegJ3SerialNumber" value="v_c_006" />
+    <xacro:property name="rightLegJ4SerialNumber" value="v_d_006" />
+    <xacro:property name="rightAnkleRightActuatorSerialNumber" value="v_e_008" />
+    <xacro:property name="rightAnkleLeftActuatorSerialNumber" value="v_e_007" />
     <xacro:property name="leftArmJ1SerialNumber" value="v_a_019" />
     <xacro:property name="leftArmJ2SerialNumber" value="v_b_014" />

Commit message: correcting rlj2 serial

File: common/xacro/serial_numbers/valkyrie_A_serials.xacro (robot description, xacro)
@@ -7,5 +7,5 @@
         <xacro:property name="leftAnkleRightActuatorSerialNumber" value="v_e_015" />
 	<xacro:property name="rightLegJ1SerialNumber" value="v_a_003" />
-        <xacro:property name="rightLegJ2SerialNumber" value="v_b_015" />
+        <xacro:property name="rightLegJ2SerialNumber" value="v_b_017" />
         <xacro:property name="rightLegJ3SerialNumber" value="v_c_009" />
         <xacro:property name="rightLegJ4SerialNumber" value="v_d_009" />
