Commit message: updated to have fpga firmware

File: common/xacro/firmware/valkyrie_firmware.xacro (robot description, xacro)
@@ -2,12 +2,17 @@
 <robot name="valkyrie_firmware_locations" xmlns:xacro="http://www.ros.org/wiki/xacro">
     <xacro:property name="PublicProcFirmwareBaseURL" value="http://linkthatdoesnotresolve.com"/>
-    <xacro:property name="PrivateProcFirmwareBaseURL" value="http://flexo.jsc.nasa.gov/bamboo/browse/DRCE-TURBOPROC/latest/artifact/shared/"/>
-    <xacro:property name="PublicFPGAFirmwareBaseURL" value="NA"/>
-    <xacro:property name="PrivateFPGAFirmwareBaseURL" value="NA"/>
+    <xacro:property name="PrivateProcFirmwareBaseURL" value="http://flexo.jsc.nasa.gov/bamboo/browse/EMB-SEAP/latest/artifact/shared/"/>
+    <xacro:property name="PublicFPGAFirmwareBaseURL" value="http://linkthatdoesnotresolve.com"/>
+    <xacro:property name="PrivateFPGAFirmwareBaseURL" value="http://flexo.jsc.nasa.gov/bamboo/browse/EMB-TURD/latest/artifact/shared/"/>
     <xacro:property name="TurboProcRotaryFirmwareExtension" value="Rotary-Binary-for-Bootloader/turbo_bootloader.bin"/>
     <xacro:property name="TurboProcLinearFirmwareExtension" value="Linear-Binary-for-Bootloader/turbo_bootloader.bin"/>
-    <xacro:property name="TurboProcRotaryFirmwareURL" value="${TurboProcRotaryFirmwareExtension}"/>
-    <xacro:property name="TurboProcLinearFirmwareURL" value="${TurboProcLinearFirmwareExtension}"/>
-    <xacro:property name="TurboFPGAFirmwareURL" value="NA"/>
+    <xacro:property name="TurboFPGAFirmwareNode1Extension" value="V1_turbodriver_daria1_c0n1.sbf.gz"/>
+    <xacro:property name="TurboFPGAFirmwareNode2Extension" value="V1_turbodriver_daria1_c0n2.sbf.gz"/>
+    <xacro:property name="TurboFPGAFirmwareNode3Extension" value="V1_turbodriver_daria1_c0n3.sbf.gz"/>
+    <xacro:property name="TurboFPGAFirmwareNode4Extension" value="V1_turbodriver_daria1_c0n4.sbf.gz"/>
+    <xacro:property name="TurboFPGAFirmwareNode5Extension" value="V1_turbodriver_daria1_c0n5.sbf.gz"/>
+    <xacro:property name="TurboFPGAFirmwareNode6Extension" value="V1_turbodriver_daria1_c0n6.sbf.gz"/>
+    <xacro:property name="TurboFPGAFirmwareNode7Extension" value="V1_turbodriver_daria1_c0n7.sbf.gz"/>
+    <xacro:property name="TurboFPGAFirmwareNode8Extension" value="V1_turbodriver_daria1_c0n8.sbf.gz"/>
     <xacro:macro name="firmware_base_url" >
         <TurbodriverProcessorFirmware>
@@ -20,26 +25,30 @@
         </TurbodriverFPGAFirmware>
     </xacro:macro>
-    <xacro:property name="HipYawProcFirmware" value="${TurboProcRotaryFirmwareURL}" />
-    <xacro:property name="HipYawFPGAFirmware" value="${TurboFPGAFirmwareURL}" />
-    <xacro:property name="HipRollProcFirmware" value="${TurboProcRotaryFirmwareURL}" />
-    <xacro:property name="HipRollFPGAFirmware" value="${TurboFPGAFirmwareURL}" />
-    <xacro:property name="HipPitchProcFirmware" value="${TurboProcRotaryFirmwareURL}" />
-    <xacro:property name="HipPitchFPGAFirmware" value="${TurboFPGAFirmwareURL}" />
-    <xacro:property name="KneePitchProcFirmware" value="${TurboProcRotaryFirmwareURL}" />
-    <xacro:property name="KneePitchFPGAFirmware" value="${TurboFPGAFirmwareURL}" />
-    <xacro:property name="AnkleLeftActuatorProcFirmware" value="${TurboProcLinearFirmwareURL}" />
-    <xacro:property name="AnkleLeftActuatorFPGAFirmware" value="${TurboFPGAFirmwareURL}" />
-    <xacro:property name="AnkleRightActuatorProcFirmware" value="${TurboProcLinearFirmwareURL}" />
-    <xacro:property name="AnkleRightActuatorFPGAFirmware" value="" />
-    <xacro:property name="ShoulderPitchProcFirmware" value="${TurboProcRotaryFirmwareURL}" />
-    <xacro:property name="ShoulderPitchFPGAFirmware" value="${TurboFPGAFirmwareURL}" />
-    <xacro:property name="ShoulderRollProcFirmware" value="${TurboProcRotaryFirmwareURL}" />
-    <xacro:property name="ShoulderRollFPGAFirmware" value="${TurboFPGAFirmwareURL}" />
-    <xacro:property name="ShoulderYawProcFirmware" value="${TurboProcRotaryFirmwareURL}" />
-    <xacro:property name="ShoulderYawFPGAFirmware" value="${TurboFPGAFirmwareURL}" />
-    <xacro:property name="ElbowPitchProcFirmware" value="${TurboProcRotaryFirmwareURL}" />
-    <xacro:property name="ElbowPitchFPGAFirmware" value="${TurboFPGAFirmwareURL}" />
-    <xacro:property name="ForearmYawProcFirmware" value="${TurboFPGAFirmwareURL}" />
-    <xacro:property name="ForearmYawFPGAFirmware" value="${TurboFPGAFirmwareURL}" />
+    <xacro:property name="LeftHipYawProcFirmware" value="${TurboProcRotaryFirmwareExtension}" />
+    <xacro:property name="LeftHipYawFPGAFirmware" value="${TurboFPGAFirmwareNode3Extension}" />
+    <xacro:property name="RightHipYawProcFirmware" value="${TurboProcRotaryFirmwareExtension}" />
+    <xacro:property name="RightHipYawFPGAFirmware" value="${TurboFPGAFirmwareNode5Extension}" />
+    <xacro:property name="HipRollProcFirmware" value="${TurboProcRotaryFirmwareExtension}" />
+    <xacro:property name="HipRollFPGAFirmware" value="${TurboFPGAFirmwareNode2Extension}" />
+    <xacro:property name="HipPitchProcFirmware" value="${TurboProcRotaryFirmwareExtension}" />
+    <xacro:property name="HipPitchFPGAFirmware" value="${TurboFPGAFirmwareNode3Extension}" />
+    <xacro:property name="KneePitchProcFirmware" value="${TurboProcRotaryFirmwareExtension}" />
+    <xacro:property name="KneePitchFPGAFirmware" value="${TurboFPGAFirmwareNode4Extension}" />
+    <xacro:property name="AnkleRightActuatorProcFirmware" value="${TurboProcLinearFirmwareExtension}" />
+    <xacro:property name="AnkleRightActuatorFPGAFirmware" value="${TurboFPGAFirmwareNode5Extension}" />
+    <xacro:property name="AnkleLeftActuatorProcFirmware" value="${TurboProcLinearFirmwareExtension}" />
+    <xacro:property name="AnkleLeftActuatorFPGAFirmware" value="${TurboFPGAFirmwareNode6Extension}" />
+    <xacro:property name="LeftShoulderPitchProcFirmware" value="${TurboProcRotaryFirmwareExtension}" />
+    <xacro:property name="LeftShoulderPitchFPGAFirmware" value="${TurboFPGAFirmwareNode1Extension}" />
+    <xacro:property name="RightShoulderPitchProcFirmware" value="${TurboProcRotaryFirmwareExtension}" />
+    <xacro:property name="RightShoulderPitchFPGAFirmware" value="${TurboFPGAFirmwareNode4Extension}" />
+    <xacro:property name="ShoulderRollProcFirmware" value="${TurboProcRotaryFirmwareExtension}" />
+    <xacro:property name="ShoulderRollFPGAFirmware" value="${TurboFPGAFirmwareNode2Extension}" />
+    <xacro:property name="ShoulderYawProcFirmware" value="${TurboProcRotaryFirmwareExtension}" />
+    <xacro:property name="ShoulderYawFPGAFirmware" value="${TurboFPGAFirmwareNode3Extension}" />
+    <xacro:property name="ElbowPitchProcFirmware" value="${TurboProcRotaryFirmwareExtension}" />
+    <xacro:property name="ElbowPitchFPGAFirmware" value="${TurboFPGAFirmwareNode4Extension}" />
+    <xacro:property name="ForearmYawProcFirmware" value="" />
+    <xacro:property name="ForearmYawFPGAFirmware" value="" />
     <xacro:property name="LowerNeckPitchProcessorFirmware" value="" />
     <xacro:property name="LowerNeckPitchFPGAFirmware" value="" />
@@ -48,10 +57,10 @@
     <xacro:property name="UpperNeckPitchProcessorFirmware" value="" />
     <xacro:property name="UpperNeckPitchFPGAFirmware" value="" />
-    <xacro:property name="TrunkYawProcessorFirmware" value="${TurboProcRotaryFirmwareURL}" />
-    <xacro:property name="TrunkYawFPGAFirmware" value="${TurboFPGAFirmwareURL}" />
-    <xacro:property name="WaistRightActuatorProcessorFirmware" value="${TurboProcLinearFirmwareURL}" />
-    <xacro:property name="WaistRightActuatorFPGAFirmware" value="${TurboFPGAFirmwareURL}" />
-    <xacro:property name="WaistLeftActuatorProcessorFirmware" value="${TurboProcLinearFirmwareURL}" />
-    <xacro:property name="WaistLeftActuatorFPGAFirmware" value="${TurboFPGAFirmwareURL}" />
+    <xacro:property name="TrunkYawProcessorFirmware" value="${TurboProcRotaryFirmwareExtension}" />
+    <xacro:property name="TrunkYawFPGAFirmware" value="${TurboFPGAFirmwareNode1Extension}" />
+    <xacro:property name="WaistLeftActuatorProcessorFirmware" value="${TurboProcLinearFirmwareExtension}" />
+    <xacro:property name="WaistLeftActuatorFPGAFirmware" value="${TurboFPGAFirmwareNode2Extension}" />
+    <xacro:property name="WaistRightActuatorProcessorFirmware" value="${TurboProcLinearFirmwareExtension}" />
+    <xacro:property name="WaistRightActuatorFPGAFirmware" value="${TurboFPGAFirmwareNode3Extension}" />
     <xacro:property name="leftForearmProcessorFirmware" value=""/>
     <xacro:property name="leftForearmFPGAFirmware" value=""/>

File: instance/instances/robots/xacro/common/valkyrie_full_template.xacro (robot description, xacro)
@@ -11,8 +11,8 @@
 	<xacro:firmware_base_url/>
 	<Mechanisms>
-		<xacro:leg prefix="left" j1_serial_number="${leftLegJ1SerialNumber}" j2_serial_number="${leftLegJ2SerialNumber}" j3_serial_number="${leftLegJ3SerialNumber}" j4_serial_number="${leftLegJ4SerialNumber}" ankle_left_actuator_serial="${leftAnkleLeftActuatorSerialNumber}" ankle_right_actuator_serial="${leftAnkleRightActuatorSerialNumber}"/>
-		<xacro:leg prefix="right" j1_serial_number="${rightLegJ1SerialNumber}" j2_serial_number="${rightLegJ2SerialNumber}" j3_serial_number="${rightLegJ3SerialNumber}" j4_serial_number="${rightLegJ4SerialNumber}" ankle_left_actuator_serial="${rightAnkleLeftActuatorSerialNumber}" ankle_right_actuator_serial="${rightAnkleRightActuatorSerialNumber}" />
-		<xacro:arm prefix="left" j1_serial_number="${leftArmJ1SerialNumber}" j2_serial_number="${leftArmJ2SerialNumber}" j3_serial_number="${leftArmJ3SerialNumber}" j4_serial_number="${leftArmJ4SerialNumber}" j5_serial_number="${leftArmJ5SerialNumber}" forearm_serial_number="${leftForearmSerialNumber}" />
-		<xacro:arm prefix="right" j1_serial_number="${rightArmJ1SerialNumber}" j2_serial_number="${rightArmJ2SerialNumber}" j3_serial_number="${rightArmJ3SerialNumber}" j4_serial_number="${rightArmJ4SerialNumber}" j5_serial_number="${rightArmJ5SerialNumber}" forearm_serial_number="${rightForearmSerialNumber}" />
+		<xacro:leg prefix="left" left_side="true" j1_serial_number="${leftLegJ1SerialNumber}" j2_serial_number="${leftLegJ2SerialNumber}" j3_serial_number="${leftLegJ3SerialNumber}" j4_serial_number="${leftLegJ4SerialNumber}" ankle_left_actuator_serial="${leftAnkleLeftActuatorSerialNumber}" ankle_right_actuator_serial="${leftAnkleRightActuatorSerialNumber}"/>
+		<xacro:leg prefix="right" left_side="false" j1_serial_number="${rightLegJ1SerialNumber}" j2_serial_number="${rightLegJ2SerialNumber}" j3_serial_number="${rightLegJ3SerialNumber}" j4_serial_number="${rightLegJ4SerialNumber}" ankle_left_actuator_serial="${rightAnkleLeftActuatorSerialNumber}" ankle_right_actuator_serial="${rightAnkleRightActuatorSerialNumber}" />
+		<xacro:arm prefix="left" left_side="true" j1_serial_number="${leftArmJ1SerialNumber}" j2_serial_number="${leftArmJ2SerialNumber}" j3_serial_number="${leftArmJ3SerialNumber}" j4_serial_number="${leftArmJ4SerialNumber}" j5_serial_number="${leftArmJ5SerialNumber}" forearm_serial_number="${leftForearmSerialNumber}" />
+		<xacro:arm prefix="right" left_side="false" j1_serial_number="${rightArmJ1SerialNumber}" j2_serial_number="${rightArmJ2SerialNumber}" j3_serial_number="${rightArmJ3SerialNumber}" j4_serial_number="${rightArmJ4SerialNumber}" j5_serial_number="${rightArmJ5SerialNumber}" forearm_serial_number="${rightForearmSerialNumber}" />
 		<xacro:neck j1_serial_number="${neckJ1SerialNumber}" j2_serial_number="${neckJ2SerialNumber}" j3_serial_number="${neckJ3SerialNumber}" />
 		<xacro:waist j1_serial_number="${trunkSerialNumber}" waist_left_actuator_serial="${waistLeftActuatorSerialNumber}" waist_right_actuator_serial="${waistRightActuatorSerialNumber}"/>

File: instance/instances/robots/xacro/limbs/arm.xacro (robot description, xacro)
@@ -3,6 +3,11 @@
     <xacro:include filename="$(find val_description)/common/xacro/joint_names/valkyrie_joint_names.xacro"/>
     <xacro:include filename="$(find val_description)/common/xacro/firmware/valkyrie_firmware.xacro"/>
-    <xacro:macro name="arm" params="prefix j1_serial_number j2_serial_number j3_serial_number j4_serial_number j5_serial_number forearm_serial_number" >
-    	<xacro:simple_mechanism name="${ShoulderPitchJointName}" serial_number="${j1_serial_number}" node="${ShoulderPitchNode}" processor_firmware="${ShoulderPitchProcFirmware}" fpga_firmware="${ShoulderPitchFPGAFirmware}"/>
+    <xacro:macro name="arm" params="prefix left_side j1_serial_number j2_serial_number j3_serial_number j4_serial_number j5_serial_number forearm_serial_number" >
+        <xacro:if value="${left_side}">$
+    	    <xacro:simple_mechanism name="${ShoulderPitchJointName}" serial_number="${j1_serial_number}" node="${ShoulderPitchNode}" processor_firmware="${LeftShoulderPitchProcFirmware}" fpga_firmware="${LeftShoulderPitchFPGAFirmware}"/>
+        </xacro:if>
+        <xacro:unless value="${left_side}">$
+    	    <xacro:simple_mechanism name="${ShoulderPitchJointName}" serial_number="${j1_serial_number}" node="${ShoulderPitchNode}" processor_firmware="${RightShoulderPitchProcFirmware}" fpga_firmware="${RightShoulderPitchFPGAFirmware}"/>
+        </xacro:unless>
     	<xacro:simple_mechanism name="${ShoulderRollJointName}" serial_number="${j2_serial_number}" node="${ShoulderRollNode}" processor_firmware="${ShoulderRollProcFirmware}" fpga_firmware="${ShoulderRollFPGAFirmware}"/>
     	<xacro:simple_mechanism name="${ShoulderYawJointName}" serial_number="${j3_serial_number}" node="${ShoulderYawNode}" processor_firmware="${ShoulderYawProcFirmware}" fpga_firmware="${ShoulderYawFPGAFirmware}"/>

File: instance/instances/robots/xacro/limbs/leg.xacro (robot description, xacro)
@@ -2,6 +2,11 @@
     <xacro:include filename="$(find val_description)/instance/instances/robots/xacro/mechanisms/mechanisms.xacro"/>
     <xacro:include filename="$(find val_description)/common/xacro/joint_names/valkyrie_joint_names.xacro"/>
-    <xacro:macro name="leg" params="prefix j1_serial_number j2_serial_number j3_serial_number j4_serial_number ankle_left_actuator_serial ankle_right_actuator_serial" >
-    	<xacro:simple_mechanism name="${HipYawJointName}" serial_number="${j1_serial_number}" node="${HipYawNode}" processor_firmware="${HipYawProcFirmware}" fpga_firmware="${HipYawFPGAFirmware}"/>
+    <xacro:macro name="leg" params="prefix left_side j1_serial_number j2_serial_number j3_serial_number j4_serial_number ankle_left_actuator_serial ankle_right_actuator_serial" >
+        <xacro:if value="${left_side}">$
+    	    <xacro:simple_mechanism name="${HipYawJointName}" serial_number="${j1_serial_number}" node="${HipYawNode}" processor_firmware="${LeftHipYawProcFirmware}" fpga_firmware="${LeftHipYawFPGAFirmware}"/>
+        </xacro:if>
+        <xacro:unless value="${left_side}">$
+    	    <xacro:simple_mechanism name="${HipYawJointName}" serial_number="${j1_serial_number}" node="${HipYawNode}" processor_firmware="${RightHipYawProcFirmware}" fpga_firmware="${RightHipYawFPGAFirmware}"/>
+        </xacro:unless>
     	<xacro:simple_mechanism name="${HipRollJointName}" serial_number="${j2_serial_number}" node="${HipRollNode}" processor_firmware="${HipRollProcFirmware}" fpga_firmware="${HipRollFPGAFirmware}"/>
     	<xacro:simple_mechanism name="${HipPitchJointName}" serial_number="${j3_serial_number}" node="${HipPitchNode}" processor_firmware="${HipPitchProcFirmware}" fpga_firmware="${HipPitchFPGAFirmware}"/>

Commit message: updated link to FPGA sbf's

File: common/xacro/firmware/valkyrie_firmware.xacro (robot description, xacro)
@@ -4,5 +4,5 @@
     <xacro:property name="PrivateProcFirmwareBaseURL" value="http://flexo.jsc.nasa.gov/bamboo/browse/EMB-SEAP/latest/artifact/shared/"/>
     <xacro:property name="PublicFPGAFirmwareBaseURL" value="http://linkthatdoesnotresolve.com"/>
-    <xacro:property name="PrivateFPGAFirmwareBaseURL" value="http://flexo.jsc.nasa.gov/bamboo/browse/EMB-TURD/latest/artifact/shared/"/>
+    <xacro:property name="PrivateFPGAFirmwareBaseURL" value="http://flexo.jsc.nasa.gov/bamboo/browse/EMB-TURD/latest/artifact/BS/SBF-File/"/>
     <xacro:property name="TurboProcRotaryFirmwareExtension" value="Rotary-Binary-for-Bootloader/turbo_bootloader.bin"/>
     <xacro:property name="TurboProcLinearFirmwareExtension" value="Linear-Binary-for-Bootloader/turbo_bootloader.bin"/>
