Commit message: modifying transmission type name

File: model/robots/common/xacro/config/valkyrie_A_transmissions.xacro (robot description, xacro)
@@ -1,5 +1,5 @@
 <?xml version="1.0" ?>
 <robot name="valkyrie_transmissions" xmlns:xacro="http://www.ros.org/wiki/xacro">
-	<xacro:property name="TorsoTransmissionType" value="robot_transmission_interface::TorsoPushrodTransmissionLoader"/>
-	<xacro:property name="AnkleTransmissionType" value="robot_transmission_interface::AnklePushrodTransmissionLoader"/>
+	<xacro:property name="TorsoTransmissionType" value="robot_transmission_interface/TorsoPushrodTransmissionLoader"/>
+	<xacro:property name="AnkleTransmissionType" value="robot_transmission_interface/AnklePushrodTransmissionLoader"/>
 </robot>

File: model/robots/common/xacro/config/valkyrie_B_transmissions.xacro (robot description, xacro)
@@ -1,5 +1,5 @@
 <?xml version="1.0" ?>
 <robot name="valkyrie_transmissions" xmlns:xacro="http://www.ros.org/wiki/xacro">
-	<xacro:property name="TorsoTransmissionType" value="robot_transmission_interface::TorsoPushrodTransmissionLoader"/>
-	<xacro:property name="AnkleTransmissionType" value="robot_transmission_interface::AnklePushrodTransmissionLoader"/>
+	<xacro:property name="TorsoTransmissionType" value="robot_transmission_interface/TorsoPushrodTransmissionLoader"/>
+	<xacro:property name="AnkleTransmissionType" value="robot_transmission_interface/AnklePushrodTransmissionLoader"/>
 </robot>

Commit message: corrected name of transmission

File: model/robots/common/xacro/config/valkyrie_A_transmissions.xacro (robot description, xacro)
@@ -1,5 +1,5 @@
 <?xml version="1.0" ?>
 <robot name="valkyrie_transmissions" xmlns:xacro="http://www.ros.org/wiki/xacro">
-	<xacro:property name="TorsoTransmissionType" value="robot_transmission_interface/TorsoPushrodTransmissionLoader"/>
-	<xacro:property name="AnkleTransmissionType" value="robot_transmission_interface/AnklePushrodTransmissionLoader"/>
+	<xacro:property name="TorsoTransmissionType" value="robot_transmission_interface/TorsoPushrodTransmission"/>
+	<xacro:property name="AnkleTransmissionType" value="robot_transmission_interface/AnklePushrodTransmission"/>
 </robot>
