Commit message: instance file loads midas coeffs - working build

File: common/xacro/nodes/forearm_testbench_nodes.xacro (robot description, xacro)
@@ -9,3 +9,4 @@
     <xacro:property name="WristLeftNode" value="/right_arm/wrist/left_actuator" />
     <xacro:property name="WristRightNode" value="/right_arm/wrist/right_actuator" />
+    <xacro:property name="ForearmSensorsNode" value="/right_arm/forearm_sensors" />
 </robot>

File: common/xacro/nodes/valkyrie_nodes.xacro (robot description, xacro)
@@ -15,4 +15,5 @@
 	<xacro:property name="WristLeftActuatorNode" value="/${prefix}_arm/wrist/left_actuator" />
 	<xacro:property name="WristRightActuatorNode" value="/${prefix}_arm/wrist/right_actuator" />
+	<xacro:property name="ForearmSensorsNode" value="/${prefix}_arm/forearm_sensors" />
     	<xacro:property name="IndexNode" value="/${prefix}_arm/hand/index" />
     	<xacro:property name="MiddleNode" value="/${prefix}_arm/hand/middle" />
@@ -23,4 +24,5 @@
     	<xacro:property name="WristLeftNode" value="/${prefix}_arm/wrist/left_actuator" />
     	<xacro:property name="WristRightNode" value="/${prefix}_arm/wrist/right_actuator" />
+    	<xacro:property name="ForearmSensorsNode" value="/${prefix}_arm/forearm_sensors" />
 	<xacro:property name="LowerNeckPitchNode" value="/neck/j1" />
 	<xacro:property name="NeckYawNode" value="/neck/j2" />

File: instance/instances/robots/forearm_testbench_right.xacro (robot description, xacro)
@@ -15,5 +15,5 @@
     <Mechanisms>
     <xacro:simple_mechanism name="testbench_actuator" serial_number="${forearm_yaw_serial_number}" node="${testbench_node}" />
-    <xacro:hand_mechanism mechanism_name="${prefix}Hand" serial_number="${hand_serial_number}" index_node="${IndexNode}" middle_node="${MiddleNode}" pinky_node="${PinkyNode}" thumb_prox_node="${ThumbProxNode}" thumb_dist_node="${ThumbDistNode}" thumb_roll_node="${ThumbRollNode}" wrist_left_node="${WristLeftNode}" wrist_right_node="${WristRightNode}" />
+    <xacro:hand_mechanism mechanism_name="${prefix}Hand" serial_number="${hand_serial_number}" index_node="${IndexNode}" middle_node="${MiddleNode}" pinky_node="${PinkyNode}" thumb_prox_node="${ThumbProxNode}" thumb_dist_node="${ThumbDistNode}" thumb_roll_node="${ThumbRollNode}" wrist_left_node="${WristLeftNode}" wrist_right_node="${WristRightNode}" forearm_sensors_node="${ForearmSensorsNode}"/>
     </Mechanisms>
     <Devices>

File: instance/instances/robots/xacro/limbs/arm/arm.xacro (robot description, xacro)
@@ -8,5 +8,5 @@
     	<xacro:simple_mechanism name="${ElbowPitchJointName}" serial_number="${j4_serial_number}" node="${ElbowPitchNode}" calibration_angle="${ElbowPitchCalibrationAngle}"/>
     	<xacro:simple_mechanism name="${ForearmYawJointName}" serial_number="${j5_serial_number}" node="${ForearmYawNode}" calibration_angle="${ForearmYawCalibrationAngle}"/>
-    	<xacro:hand_mechanism mechanism_name="${prefix}Hand" serial_number="${forearm_serial_number}" index_node="${IndexNode}" middle_node="${MiddleNode}" pinky_node="${PinkyNode}" thumb_prox_node="${ThumbProxNode}" thumb_dist_node="${ThumbDistNode}" thumb_roll_node="${ThumbRollNode}" wrist_left_node="${WristLeftNode}" wrist_right_node="${WristRightNode}" />
+    	<xacro:hand_mechanism mechanism_name="${prefix}Hand" serial_number="${forearm_serial_number}" index_node="${IndexNode}" middle_node="${MiddleNode}" pinky_node="${PinkyNode}" thumb_prox_node="${ThumbProxNode}" thumb_dist_node="${ThumbDistNode}" thumb_roll_node="${ThumbRollNode}" wrist_left_node="${WristLeftNode}" wrist_right_node="${WristRightNode}" forearm_sensors_node="${ForearmSensorsNode}"/>
     </xacro:macro>
 </robot>

File: instance/instances/robots/xacro/mechanisms/mechanisms.xacro (robot description, xacro)
@@ -39,5 +39,5 @@
     </Mechanism>
 </xacro:macro>
-<xacro:macro name="hand_mechanism" params="mechanism_name serial_number index_node middle_node pinky_node thumb_prox_node thumb_dist_node thumb_roll_node wrist_left_node wrist_right_node" >
+<xacro:macro name="hand_mechanism" params="mechanism_name serial_number index_node middle_node pinky_node thumb_prox_node thumb_dist_node thumb_roll_node wrist_left_node wrist_right_node forearm_sensors_node" >
     <Mechanism id="${mechanism_name}" type="hand">
             <SerialNumber id="${serial_number}"/>
@@ -51,4 +51,5 @@
                 <WristLeft id="${wrist_left_node}"/>
                 <WristRight id="${wrist_right_node}"/>
+                <ForearmSensors id="${forearm_sensors_node}"/>
             </Nodes>
     </Mechanism>
