Commit message: added imu urdf fot test of kvh vs microstrain

File: common/xacro/config_packages/valkyrie_imu_test_pkg.xacro (robot description, xacro)
@@ -1,4 +1,6 @@
 <robot xmlns:xacro="http://ros.org/wiki/xacro" name="valkyrie_imu_test_pkg">
 	<xacro:property name="pelvis_middle_imu_pkg" value="val_config_files" />
-	<xacro:property name="pelvis_middle_imu_cal" value="kvh_1750/1608K047/Calibration.cal" />
+	<xacro:property name="pelvis_rear_imu_pkg" value="val_config_files" />
+	<xacro:property name="pelvis_middle_imu_cal" value="kvh_1750/1608K048/Calibration.cal" />
+	<xacro:property name="pelvis_rear_imu_cal" value="3dm_gx4_15/47099/Calibration.cal" />
 </robot>

File: model/robots/common/xacro/valkyrie_imu_base.xacro (robot description, xacro)
@@ -1,6 +1,7 @@
 <robot xmlns:xacro="http://ros.org/wiki/xacro" name="valkyrie_imu_base">
-    <xacro:property name="KVHHardwareApi" value="val_imu_kvh_1750_interface/ImuKVHInterface" />
+    <xacro:property name="KVHHardwareApi" value="kvh_1750_sensor::KVH1750ConstSensor" />
+    <xacro:property name="MicroStrainHardwareApi" value="imu_3dm_gx4_15_sensor::Imu3DmGx415Sensor" />
     <xacro:make_pelvis />
     <xacro:include_multisense_hw />
-    <xacro:v1_pelvis_middle_sensors_usb sensor_node_tag="${pelvis_middle_imu_node}" sensor_api_tag="${KVHHardwareApi}"  sensor_pkg_tag="${pelvis_middle_imu_pkg}" sensor_config_tag="${pelvis_middle_imu_cal}" />
+    <xacro:v1_pelvis_sensors_usb middle_sensor_node_tag="${pelvis_middle_imu_node}" middle_sensor_api_tag="${KVHHardwareApi}" middle_sensor_pkg_tag="${pelvis_middle_imu_pkg}" middle_sensor_config_tag="${pelvis_middle_imu_cal}" rear_sensor_node_tag="${pelvis_rear_imu_node}" rear_sensor_api_tag="${MicroStrainHardwareApi}" rear_sensor_pkg_tag="${pelvis_rear_imu_pkg}" rear_sensor_config_tag="${pelvis_rear_imu_cal}"/>
 </robot>

Commit message: updating imu testing xacros

File: common/xacro/config_packages/valkyrie_imu_test_pkg.xacro (robot description, xacro)
@@ -2,5 +2,7 @@
 	<xacro:property name="pelvis_middle_imu_pkg" value="val_config_files" />
 	<xacro:property name="pelvis_rear_imu_pkg" value="val_config_files" />
+	<xacro:property name="pelvis_test_imu_pkg" value="val_config_files" />
 	<xacro:property name="pelvis_middle_imu_cal" value="kvh_1750/1608K048/Calibration.cal" />
 	<xacro:property name="pelvis_rear_imu_cal" value="3dm_gx4_15/47099/Calibration.cal" />
+	<xacro:property name="pelvis_test_imu_cal" value="stim300/N25581710875719/Calibration.cal" />
 </robot>

File: model/robots/common/xacro/valkyrie_imu_base.xacro (robot description, xacro)
@@ -2,7 +2,8 @@
     <xacro:property name="KVHHardwareApi" value="kvh_1750_sensor::KVH1750ConstSensor" />
     <xacro:property name="MicroStrainHardwareApi" value="imu_3dm_gx4_15_sensor::Imu3DmGx415Sensor" />
+    <xacro:property name="StimHardwareApi" value="stim_300_sensor::STIM300ConstSensor" />
     <xacro:make_pelvis />
     <xacro:include_multisense_hw />
     <!-- <xacro:v1_pelvis_sensors_usb middle_sensor_node_tag="${pelvis_middle_imu_node}" middle_sensor_api_tag="${KVHHardwareApi}" middle_sensor_pkg_tag="${pelvis_middle_imu_pkg}" middle_sensor_config_tag="${pelvis_middle_imu_cal}" rear_sensor_node_tag="${pelvis_rear_imu_node}" rear_sensor_api_tag="${MicroStrainHardwareApi}" rear_sensor_pkg_tag="${pelvis_rear_imu_pkg}" rear_sensor_config_tag="${pelvis_rear_imu_cal}"/> -->
-    <xacro:v1_pelvis_middle_sensors_usb sensor_node_tag="${pelvis_middle_imu_node}" sensor_api_tag="${KVHHardwareApi}" sensor_pkg_tag="${pelvis_middle_imu_pkg}" sensor_config_tag="${pelvis_middle_imu_cal}" />
+    <xacro:v1_pelvis_middle_sensors_usb sensor_node_tag="${pelvis_middle_imu_node}" sensor_api_tag="${KVHHardwareApi}" sensor_pkg_tag="${pelvis_test_imu_pkg}" sensor_config_tag="${pelvis_test_imu_cal}" />
 </robot>
