Commit message: updated to use package and file rather than port numbers and serial numbers to prevent hard coded file paths

File: common/xacro/config_packages/valkyrie_A_pkg.xacro (robot description, xacro)
@@ -2,6 +2,11 @@
 	<xacro:property name="left_foot_ATI_pkg" value="val_config_files" />
 	<xacro:property name="right_foot_ATI_pkg" value="val_config_files" />
+	<xacro:property name="left_foot_ATI_cal" value="ati_config/FT17218.cal"/>
+	<xacro:property name="right_foot_ATI_cal" value="ati_config/FT16592.cal" />
 	<xacro:property name="pelvis_middle_imu_pkg" value="val_config_files" />
 	<xacro:property name="pelvis_rear_imu_pkg" value="val_config_files" />
 	<xacro:property name="torso_left_imu_pkg" value="val_config_files" />
+	<xacro:property name="pelvis_middle_imu_cal" value="None" />
+	<xacro:property name="pelvis_rear_imu_cal" value="3dm_gx4_15/47090/Calibration.cal" />
+	<xacro:property name="torso_left_imu_cal" value="3dm_gx4_15/47095/Calibration.cal" />
 </robot>

File: common/xacro/config_packages/valkyrie_B_pkg.xacro (robot description, xacro)
@@ -1,7 +1,12 @@
-<robot xmlns:xacro="http://ros.org/wiki/xacro" name="valkyrie_A_pkg">
+<robot xmlns:xacro="http://ros.org/wiki/xacro" name="valkyrie_B_pkg">
 	<xacro:property name="left_foot_ATI_pkg" value="val_config_files" />
 	<xacro:property name="right_foot_ATI_pkg" value="val_config_files" />
+	<xacro:property name="left_foot_ATI_cal" value="ati_config/FT16594.cal"/>
+	<xacro:property name="right_foot_ATI_cal" value="ati_config/FT14018.cal" />
 	<xacro:property name="pelvis_middle_imu_pkg" value="val_config_files" />
 	<xacro:property name="pelvis_rear_imu_pkg" value="val_config_files" />
 	<xacro:property name="torso_left_imu_pkg" value="val_config_files" />
+	<xacro:property name="pelvis_middle_imu_cal" value="3dm_gx4_15/47094/Calibration.cal" />
+	<xacro:property name="pelvis_rear_imu_cal" value="3dm_gx4_15/47092/Calibration.cal" />
+	<xacro:property name="torso_left_imu_cal" value="3dm_gx4_15/47097/Calibration.cal" />
 </robot>

File: common/xacro/config_packages/valkyrie_C_pkg.xacro (robot description, xacro)
@@ -1,7 +1,12 @@
-<robot xmlns:xacro="http://ros.org/wiki/xacro" name="valkyrie_A_pkg">
+<robot xmlns:xacro="http://ros.org/wiki/xacro" name="valkyrie_C_pkg">
 	<xacro:property name="left_foot_ATI_pkg" value="val_config_files" />
 	<xacro:property name="right_foot_ATI_pkg" value="val_config_files" />
+	<xacro:property name="left_foot_ATI_cal" value="ati_config/FT14020.cal"/>
+	<xacro:property name="right_foot_ATI_cal" value="ati_config/FT17214.cal" />
 	<xacro:property name="pelvis_middle_imu_pkg" value="val_config_files" />
 	<xacro:property name="pelvis_rear_imu_pkg" value="val_config_files" />
 	<xacro:property name="torso_left_imu_pkg" value="val_config_files" />
+	<xacro:property name="pelvis_middle_imu_cal" value="None" />
+	<xacro:property name="pelvis_rear_imu_cal" value="3dm_gx4_15/47250/Calibration.cal" />
+	<xacro:property name="torso_left_imu_cal" value="3dm_gx4_15/47096/Calibration.cal" />
 </robot>

File: common/xacro/config_packages/valkyrie_gazebo_pkg.xacro (robot description, xacro)
@@ -1,12 +1,12 @@
-<robot xmlns:xacro="http://ros.org/wiki/xacro" name="valkyrie_D_pkg">
+<robot xmlns:xacro="http://ros.org/wiki/xacro" name="valkyrie_gazebo_pkg">
 	<xacro:property name="left_foot_ATI_pkg" value="val_config_files" />
 	<xacro:property name="right_foot_ATI_pkg" value="val_config_files" />
-	<xacro:property name="left_foot_ATI_cal" value="ati_config/FT17212.cal"/>
-	<xacro:property name="right_foot_ATI_cal" value="ati_config/FT16590.cal" />
+	<xacro:property name="left_foot_ATI_cal" value="ati_config/FT001SIM.cal"/>
+	<xacro:property name="right_foot_ATI_cal" value="ati_config/FT001SIM.cal" />
 	<xacro:property name="pelvis_middle_imu_pkg" value="val_config_files" />
 	<xacro:property name="pelvis_rear_imu_pkg" value="val_config_files" />
 	<xacro:property name="torso_left_imu_pkg" value="val_config_files" />
 	<xacro:property name="pelvis_middle_imu_cal" value="None" />
-	<xacro:property name="pelvis_rear_imu_cal" value="3dm_gx4_15/51067/Calibration.cal" />
-	<xacro:property name="torso_left_imu_cal" value="3dm_gx4_15/47093/Calibration.cal" />
+	<xacro:property name="pelvis_rear_imu_cal" value="None" />
+	<xacro:property name="torso_left_imu_cal" value="None" />
 </robot>

File: model/robots/common/xacro/leg/leg.xacro (robot description, xacro)
@@ -147,5 +147,5 @@
     <xacro:make_ankle_joints prefix="${prefix}" reflect="${reflect}" leg_root_link="${leg_root_link}" />
   </xacro:macro>
-  <xacro:macro name="v1_leg_sensors" params="prefix reflect ATI_serial_number ATI_node">
+  <xacro:macro name="v1_leg_sensors" params="prefix reflect ATI_node ATI_sensor_pkg ATI_config_file">
     <xacro:virtual_fixed_frame_offset name="${prefix}COP"
                        parentLink="${AnkleRollLinkName}"
@@ -157,7 +157,8 @@
                         origin_xyz="0.0215646 0.0 -0.051054"
                         origin_rpy="3.14 0.0 0.0"
-                        sensor_number="${ATI_serial_number}"
                         sensor_node="${ATI_node}"
-                        sensor_api="${ForceTorqueSensorApi}" />
+                        sensor_api="${ForceTorqueSensorApi}"
+                        sensor_pkg="${ATI_sensor_pkg}"
+                        sensor_config_file="${ATI_config_file}" />
   </xacro:macro>
   <xacro:macro name="leg_transmissions_hw" params="prefix">

File: model/robots/common/xacro/pelvis/pelvis.xacro (robot description, xacro)
@@ -12,19 +12,19 @@
     </xacro:macro>
     <xacro:macro name="v1_pelvis_sensors">
-        <xacro:microstrain_sensor sensorName="pelvisRearImu"
+        <xacro:imu_sensor sensorName="pelvisRearImu"
                                   parentLink="${Pelvis_Link_Name}"
                                   origin_xyz="-0.075844901 0.0 -0.111056426"
                                   origin_rpy="-3.14159 0.476467 -3.14159" />
-        <xacro:microstrain_sensor sensorName="pelvisMiddleImu"
+        <xacro:imu_sensor sensorName="pelvisMiddleImu"
                                   parentLink="${Pelvis_Link_Name}"
                                   origin_xyz="0.150 0.0 0.08"
                                   origin_rpy="0.0 0.0 0.7854" />
     </xacro:macro>
-    <xacro:macro name="v1_pelvis_middle_sensors_usb" params="sensor_node_tag sensor_api_tag sensor_port_tag">
-        <xacro:microstrain_sensor sensorName="pelvisRearImu"
+    <xacro:macro name="v1_pelvis_middle_sensors_usb" params="sensor_node_tag sensor_api_tag sensor_pkg_tag sensor_config_tag">
+        <xacro:imu_sensor sensorName="pelvisRearImu"
                                   parentLink="${Pelvis_Link_Name}"
                                   origin_xyz="-0.075844901 0.0 -0.111056426"
                                   origin_rpy="-3.14159 0.476467 -3.14159" />
-        <xacro:usb_microstrain_sensor sensorName="pelvisMiddleImu"
+        <xacro:usb_imu_sensor sensorName="pelvisMiddleImu"
                                   parentLink="${Pelvis_Link_Name}"
                                   origin_xyz="0.0 0.0 -0.10819638"
@@ -32,8 +32,9 @@
                                   sensor_node="${sensor_node_tag}"
                                   sensor_api="${sensor_api_tag}"
-                                  sensor_port="${sensor_port_tag}" />
+                                  sensor_pkg="${sensor_pkg_tag}"
+                                  sensor_config_file="${sensor_config_tag}" />
     </xacro:macro>
-    <xacro:macro name="v1_pelvis_rear_sensors_usb" params="sensor_node_tag sensor_api_tag sensor_port_tag">
-        <xacro:usb_microstrain_sensor sensorName="pelvisRearImu"
+    <xacro:macro name="v1_pelvis_rear_sensors_usb" params="sensor_node_tag sensor_api_tag sensor_pkg_tag sensor_config_tag">
+        <xacro:usb_imu_sensor sensorName="pelvisRearImu"
                                   parentLink="${Pelvis_Link_Name}"
                                   origin_xyz="-0.075844901 0.0 -0.111056426"
@@ -41,12 +42,13 @@
                         				  sensor_node="${sensor_node_tag}"
                         				  sensor_api="${sensor_api_tag}"
-                        				  sensor_port="${sensor_port_tag}" />
-        <xacro:microstrain_sensor sensorName="pelvisMiddleImu"
+                        				  sensor_pkg="${sensor_pkg_tag}"
+                                  sensor_config_file="${sensor_config_tag}" />
+        <xacro:imu_sensor sensorName="pelvisMiddleImu"
                                   parentLink="${Pelvis_Link_Name}"
                                   origin_xyz="0.0 0.0 -0.10819638"
                                   origin_rpy="3.14159 0.0 0.0" />
     </xacro:macro>
-    <xacro:macro name="v1_pelvis_sensors_usb" params="middle_sensor_node_tag middle_sensor_api_tag middle_sensor_port_tag rear_sensor_node_tag rear_sensor_api_tag rear_sensor_port_tag">
-        <xacro:usb_microstrain_sensor sensorName="pelvisRearImu"
+    <xacro:macro name="v1_pelvis_sensors_usb" params="middle_sensor_node_tag middle_sensor_api_tag middle_sensor_pkg_tag middle_sensor_config_tag rear_sensor_node_tag rear_sensor_api_tag rear_sensor_pkg_tag rear_sensor_config_tag">
+        <xacro:usb_imu_sensor sensorName="pelvisRearImu"
                                   parentLink="${Pelvis_Link_Name}"
                                   origin_xyz="-0.075844901 0.0 -0.111056426"
@@ -54,6 +56,7 @@
                                   sensor_node="${rear_sensor_node_tag}"
                                   sensor_api="${rear_sensor_api_tag}"
-                                  sensor_port="${rear_sensor_port_tag}" />
-        <xacro:usb_microstrain_sensor sensorName="pelvisMiddleImu"
+                                  sensor_pkg="${rear_sensor_pkg_tag}"
+                                  sensor_config_file="${rear_sensor_config_tag}" />
+        <xacro:usb_imu_sensor sensorName="pelvisMiddleImu"
                                   parentLink="${Pelvis_Link_Name}"
                                   origin_xyz="0.0 0.0 -0.10819638"
@@ -61,5 +64,6 @@
                                   sensor_node="${middle_sensor_node_tag}"
                                   sensor_api="${middle_sensor_api_tag}"
-                                  sensor_port="${middle_sensor_port_tag}" />
+                                  sensor_pkg="${middle_sensor_pkg_tag}"
+                                  sensor_config_file="${middle_sensor_config_tag}" />
     </xacro:macro>
 </robot>

File: model/robots/common/xacro/sensors/ati_force_torque.xacro (robot description, xacro)
@@ -1,5 +1,5 @@
 <?xml version="1.0" ?>
 <robot xmlns:xacro="http://www.ros.org/wiki/xacro" name="ati_force_torque_sensor">
-  <xacro:macro name="ati_force_torque_sensor" params="sensorName parentLink joint_to_attach_sensor_to origin_xyz origin_rpy sensor_number sensor_node sensor_api">
+  <xacro:macro name="ati_force_torque_sensor" params="sensorName parentLink joint_to_attach_sensor_to origin_xyz origin_rpy sensor_node sensor_api sensor_pkg sensor_config_file">
     <xacro:massless_virtual_link name="${sensorName}_Frame"
                     origin_rpy="0 0 0"
@@ -12,7 +12,8 @@
       <sensor name="${sensorName}" type="force_torque">
         <pose>${origin_xyz} ${origin_rpy}</pose>
-        <sensor_number id="${sensor_number}" />
         <node id="${sensor_node}" />
         <api name="${sensor_api}" />
+        <package name="${sensor_pkg}" />
+        <config name="${sensor_config_file}" />
         <always_on>true</always_on>
         <update_rate>500.0</update_rate>

File: model/robots/common/xacro/sensors/inertial_measurement_unit.xacro (robot description, xacro)
@@ -1,5 +1,5 @@
 <?xml version="1.0" ?>
-<robot xmlns:xacro="http://www.ros.org/wiki/xacro" name="microstrain">
-  <xacro:macro name="microstrain_sensor" params="sensorName parentLink origin_xyz origin_rpy">
+<robot xmlns:xacro="http://www.ros.org/wiki/xacro" name="inertial_measurement_unit">
+  <xacro:macro name="imu_sensor" params="sensorName parentLink origin_xyz origin_rpy">
     <xacro:massless_virtual_link name="${sensorName}_Frame"
                     origin_rpy="0 0 0"
@@ -44,5 +44,5 @@
     </gazebo>
   </xacro:macro>
-  <xacro:macro name="usb_microstrain_sensor" params="sensorName parentLink origin_xyz origin_rpy sensor_node sensor_api sensor_port">
+  <xacro:macro name="usb_imu_sensor" params="sensorName parentLink origin_xyz origin_rpy sensor_node sensor_api sensor_pkg sensor_config_file">
     <xacro:massless_virtual_link name="${sensorName}_Frame"
                     origin_rpy="0 0 0"
@@ -67,7 +67,8 @@
         <always_on>true</always_on>
         <pose>0 0 0 0 0 0 </pose>
-        <node name="${sensor_node}" />
+        <node id="${sensor_node}" />
         <api name="${sensor_api}" />
-        <port name="${sensor_port}" />
+        <package name="${sensor_pkg}" />
+        <config name="${sensor_config_file}" />
         <imu>
            <noise>

File: model/robots/common/xacro/valkyrie_arm_mass_sims_base_hw.xacro (robot description, xacro)
@@ -7,9 +7,9 @@
     <xacro:make_leg prefix="right" reflect="-1" leg_root_link="${Pelvis_Link_Name}"/>
     <xacro:make_leg prefix="left" reflect="1" leg_root_link="${Pelvis_Link_Name}"/>
-    <xacro:v1_trunk_sensors_usb sensor_node_tag="${torso_left_imu_node}" sensor_api_tag="${ImuMicrostrainHardwareApi}" sensor_port_tag="${torso_left_imu_port}"/>
-    <xacro:v1_leg_sensors prefix="left" reflect="1" ATI_serial_number="${left_foot_ATI_serial}" ATI_node="${left_foot_ATI_node}"/>
-    <xacro:v1_leg_sensors prefix="right" reflect="-1" ATI_serial_number="${right_foot_ATI_serial}" ATI_node="${right_foot_ATI_node}"/>
+    <xacro:v1_trunk_sensors_usb sensor_node_tag="${torso_left_imu_node}" sensor_api_tag="${ImuMicrostrainHardwareApi}" sensor_pkg_tag="${torso_left_imu_pkg}" sensor_config_tag="${torso_left_imu_cal}" />
+    <xacro:v1_leg_sensors prefix="left" reflect="1" ATI_node="${left_foot_ATI_node}" ATI_sensor_pkg="${left_foot_ATI_pkg}" ATI_config_file="${left_foot_ATI_cal}"/>
+    <xacro:v1_leg_sensors prefix="right" reflect="-1" ATI_node="${right_foot_ATI_node}" ATI_sensor_pkg="${right_foot_ATI_pkg}" ATI_config_file="${right_foot_ATI_cal}"/>
     <xacro:include_multisense_hw />
-    <xacro:v1_pelvis_rear_sensors_usb sensor_node_tag="${pelvis_rear_imu_node}" sensor_api_tag="${ImuMicrostrainHardwareApi}"  sensor_port_tag="${pelvis_rear_imu_port}"/>
+    <xacro:v1_pelvis_rear_sensors_usb sensor_node_tag="${pelvis_rear_imu_node}" sensor_api_tag="${ImuMicrostrainHardwareApi}"  sensor_pkg_tag="${pelvis_rear_imu_pkg}" sensor_config_tag="${pelvis_rear_imu_cal}" />
     <xacro:waist_transmissions_hw />
     <xacro:leg_transmissions_hw prefix="left"/>

File: model/robots/common/xacro/valkyrie_arm_mass_sims_base_sim.xacro (robot description, xacro)
@@ -7,9 +7,9 @@
     <xacro:make_leg prefix="right" reflect="-1" leg_root_link="${Pelvis_Link_Name}"/>
     <xacro:make_leg prefix="left" reflect="1" leg_root_link="${Pelvis_Link_Name}"/>
-    <xacro:v1_pelvis_sensors_usb middle_sensor_node_tag="${pelvis_middle_imu_node}" middle_sensor_api_tag="${ImuSensorSimApi}" middle_sensor_port_tag="${pelvis_middle_imu_port}" rear_sensor_node_tag="${pelvis_rear_imu_node}" rear_sensor_api_tag="${ImuSensorSimApi}" rear_sensor_port_tag="${pelvis_rear_imu_port}"/>
-    <xacro:v1_leg_sensors prefix="left" reflect="1" ATI_serial_number="${sim_ATI_serial}" ATI_node="${left_foot_Sim_ATI_node}"/>
-    <xacro:v1_leg_sensors prefix="right" reflect="-1" ATI_serial_number="${sim_ATI_serial}" ATI_node="${right_foot_Sim_ATI_node}"/>
+    <xacro:v1_pelvis_sensors_usb middle_sensor_node_tag="${pelvis_middle_imu_node}" middle_sensor_api_tag="${ImuSensorSimApi}" middle_sensor_pkg_tag="${pelvis_middle_imu_pkg}" middle_sensor_config_tag="${pelvis_middle_imu_cal}" rear_sensor_node_tag="${pelvis_rear_imu_node}" rear_sensor_api_tag="${ImuSensorSimApi}" rear_sensor_pkg_tag="${pelvis_rear_imu_pkg}" rear_sensor_config_tag="${pelvis_rear_imu_cal}"/>
+    <xacro:v1_leg_sensors prefix="left" reflect="1" ATI_node="${left_foot_Sim_ATI_node}" ATI_sensor_pkg="${left_foot_ATI_pkg}" ATI_config_file="${left_foot_ATI_cal}"/>
+    <xacro:v1_leg_sensors prefix="right" reflect="-1" ATI_node="${right_foot_Sim_ATI_node}" ATI_sensor_pkg="${right_foot_ATI_pkg}" ATI_config_file="${right_foot_ATI_cal}"/>
     <xacro:include_multisense_sim />
-    <xacro:v1_trunk_sensors_usb sensor_node_tag="${torso_left_imu_node}" sensor_api_tag="${ImuSensorSimApi}" sensor_port_tag="${torso_left_imu_port}"/>
+    <xacro:v1_trunk_sensors_usb sensor_node_tag="${torso_left_imu_node}" sensor_api_tag="${ImuSensorSimApi}" sensor_pkg_tag="${torso_left_imu_pkg}" sensor_config_tag="${torso_left_imu_cal}" />
     <xacro:waist_transmissions_sim />
     <xacro:leg_transmissions_sim prefix="left"/>

File: model/robots/common/xacro/valkyrie_base_hw.xacro (robot description, xacro)
@@ -15,9 +15,9 @@
     <xacro:make_leg prefix="right" reflect="-1" leg_root_link="${Pelvis_Link_Name}"/>
     <xacro:make_leg prefix="left" reflect="1" leg_root_link="${Pelvis_Link_Name}"/>
-    <xacro:v1_trunk_sensors_usb sensor_node_tag="${torso_left_imu_node}" sensor_api_tag="${ImuMicrostrainHardwareApi}" sensor_port_tag="${torso_left_imu_port}"/>
-    <xacro:v1_leg_sensors prefix="left" reflect="1" ATI_serial_number="${left_foot_ATI_serial}" ATI_node="${left_foot_ATI_node}"/>
-    <xacro:v1_leg_sensors prefix="right" reflect="-1" ATI_serial_number="${right_foot_ATI_serial}" ATI_node="${right_foot_ATI_node}"/>
+    <xacro:v1_trunk_sensors_usb sensor_node_tag="${torso_left_imu_node}" sensor_api_tag="${ImuMicrostrainHardwareApi}" sensor_pkg_tag="${torso_left_imu_pkg}" sensor_config_tag="${torso_left_imu_cal}" />
+    <xacro:v1_leg_sensors prefix="left" reflect="1" ATI_node="${left_foot_ATI_node}" ATI_sensor_pkg="${left_foot_ATI_pkg}" ATI_config_file="${left_foot_ATI_cal}"/>
+    <xacro:v1_leg_sensors prefix="right" reflect="-1" ATI_node="${right_foot_ATI_node}" ATI_sensor_pkg="${right_foot_ATI_pkg}" ATI_config_file="${right_foot_ATI_cal}"/>
     <xacro:include_multisense_hw />
-    <xacro:v1_pelvis_rear_sensors_usb sensor_node_tag="${pelvis_rear_imu_node}" sensor_api_tag="${ImuMicrostrainHardwareApi}"  sensor_port_tag="${pelvis_rear_imu_port}"/>
+    <xacro:v1_pelvis_rear_sensors_usb sensor_node_tag="${pelvis_rear_imu_node}" sensor_api_tag="${ImuMicrostrainHardwareApi}"  sensor_pkg_tag="${pelvis_rear_imu_pkg}" sensor_config_tag="${pelvis_rear_imu_cal}" />
     <xacro:waist_transmissions_hw />
     <xacro:leg_transmissions_hw prefix="left"/>

File: model/robots/common/xacro/valkyrie_base_sim.xacro (robot description, xacro)
@@ -15,9 +15,9 @@
     <xacro:make_leg prefix="right" reflect="-1" leg_root_link="${Pelvis_Link_Name}"/>
     <xacro:make_leg prefix="left" reflect="1" leg_root_link="${Pelvis_Link_Name}"/>
-    <xacro:v1_pelvis_sensors_usb middle_sensor_node_tag="${pelvis_middle_imu_node}" middle_sensor_api_tag="${ImuSensorSimApi}" middle_sensor_port_tag="${pelvis_middle_imu_port}" rear_sensor_node_tag="${pelvis_rear_imu_node}" rear_sensor_api_tag="${ImuSensorSimApi}" rear_sensor_port_tag="${pelvis_rear_imu_port}"/>
-    <xacro:v1_leg_sensors prefix="left" reflect="1" ATI_serial_number="${sim_ATI_serial}" ATI_node="${left_foot_Sim_ATI_node}"/>
-    <xacro:v1_leg_sensors prefix="right" reflect="-1" ATI_serial_number="${sim_ATI_serial}" ATI_node="${right_foot_Sim_ATI_node}"/>
+    <xacro:v1_pelvis_sensors_usb middle_sensor_node_tag="${pelvis_middle_imu_node}" middle_sensor_api_tag="${ImuSensorSimApi}" middle_sensor_pkg_tag="${pelvis_middle_imu_pkg}" middle_sensor_config_tag="${pelvis_middle_imu_cal}" rear_sensor_node_tag="${pelvis_rear_imu_node}" rear_sensor_api_tag="${ImuSensorSimApi}" rear_sensor_pkg_tag="${pelvis_rear_imu_pkg}" rear_sensor_config_tag="${pelvis_rear_imu_cal}"/>
+    <xacro:v1_leg_sensors prefix="left" reflect="1" ATI_node="${left_foot_Sim_ATI_node}" ATI_sensor_pkg="${left_foot_ATI_pkg}" ATI_config_file="${left_foot_ATI_cal}"/>
+    <xacro:v1_leg_sensors prefix="right" reflect="-1" ATI_node="${right_foot_Sim_ATI_node}" ATI_sensor_pkg="${right_foot_ATI_pkg}" ATI_config_file="${right_foot_ATI_cal}"/>
     <xacro:include_multisense_sim />
-    <xacro:v1_trunk_sensors_usb sensor_node_tag="${torso_left_imu_node}" sensor_api_tag="${ImuSensorSimApi}" sensor_port_tag="${torso_left_imu_port}"/>
+    <xacro:v1_trunk_sensors_usb sensor_node_tag="${torso_left_imu_node}" sensor_api_tag="${ImuSensorSimApi}" sensor_pkg_tag="${torso_left_imu_pkg}" sensor_config_tag="${torso_left_imu_cal}" />
     <xacro:waist_transmissions_sim />
     <xacro:leg_transmissions_sim prefix="left"/>

File: model/robots/common/xacro/valkyrie_imu_base.xacro (robot description, xacro)
@@ -1,6 +1,6 @@
-<robot xmlns:xacro="http://ros.org/wiki/xacro" name="valkyrie">
+<robot xmlns:xacro="http://ros.org/wiki/xacro" name="valkyrie_imu_base">
     <xacro:property name="KVHHardwareApi" value="val_imu_kvh_1750_interface/ImuKVHInterface" />
     <xacro:make_pelvis />
     <xacro:include_multisense_hw />
-    <xacro:v1_pelvis_middle_sensors_usb sensor_node_tag="${pelvis_middle_imu_node}" sensor_api_tag="${KVHHardwareApi}"  sensor_port_tag="${pelvis_middle_imu_port}"/>
+    <xacro:v1_pelvis_middle_sensors_usb sensor_node_tag="${pelvis_middle_imu_node}" sensor_api_tag="${KVHHardwareApi}"  sensor_pkg_tag="${pelvis_middle_imu_pkg}" sensor_config_tag="${pelvis_middle_imu_cal}" />
 </robot>
