Commit message: updated to use package and file rather than port numbers and serial numbers to prevent hard coded file paths

File: model/robots/common/xacro/waist/waist.xacro (robot description, xacro)
@@ -9,5 +9,5 @@
   <xacro:include filename="$(find val_description)/model/robots/common/xacro/waist/frame_parameters.xacro"/>
   <xacro:include filename="$(find val_description)/model/robots/common/xacro/waist/mass_parameters.xacro"/>
-  <xacro:include filename="$(find val_description)/model/robots/common/xacro/sensors/microstrain.xacro"/>
+  <xacro:include filename="$(find val_description)/model/robots/common/xacro/sensors/inertial_measurement_unit.xacro"/>
   <xacro:include filename="$(find val_description)/model/robots/common/xacro/sensors/flea.xacro"/>
   <xacro:macro name="make_waist_common" params="waist_root_link">
@@ -68,5 +68,5 @@
   </xacro:macro>
   <xacro:macro name="v1_trunk_sensors">
-    <xacro:microstrain_sensor sensorName="leftTorsoImu"
+    <xacro:imu_sensor sensorName="leftTorsoImu"
                               parentLink="${TorsoRollLinkName}"
                               origin_xyz="-0.0627634 0.134239 0.3630676"
@@ -85,6 +85,6 @@
                         frameRate="60"/>
    </xacro:macro>
-  <xacro:macro name="v1_trunk_sensors_usb" params="sensor_node_tag sensor_api_tag sensor_port_tag">
-    <xacro:usb_microstrain_sensor sensorName="leftTorsoImu"
+  <xacro:macro name="v1_trunk_sensors_usb" params="sensor_node_tag sensor_api_tag sensor_pkg_tag sensor_config_tag">
+    <xacro:usb_imu_sensor sensorName="leftTorsoImu"
                               parentLink="${TorsoRollLinkName}"
                               origin_xyz="-0.0627634 0.134239 0.3630676"
@@ -92,5 +92,6 @@
                               sensor_node="${sensor_node_tag}"
                               sensor_api="${sensor_api_tag}"
-                              sensor_port="${sensor_port_tag}" />
+                              sensor_pkg="${sensor_pkg_tag}"
+                              sensor_config_file="${sensor_config_tag}" />
     <xacro:flea3_camera sensorName="rightHazardCamera"
                         parentLink="${TorsoRollLinkName}"

File: model/robots/imu_test.xacro (robot description, xacro)
@@ -1,3 +1,3 @@
-<robot xmlns:xacro="http://ros.org/wiki/xacro" name="valkyrie">
+<robot xmlns:xacro="http://ros.org/wiki/xacro" name="valkyrie_imu_test">
     <xacro:property name="mesh_root" value="package://val_description/model/meshes"/>
     <xacro:include filename="$(find val_description)/model/robots/common/xacro/generic_models.xacro" />
@@ -6,3 +6,4 @@
     <xacro:include filename="$(find val_description)/common/xacro/serial_numbers/valkyrie_C_serials.xacro"/>
     <xacro:include filename="$(find val_description)/common/xacro/dev_ports/valkyrie_imu_test_ports.xacro"/>
+    <xacro:include filename="$(find val_description)/common/xacro/config_packages/valkyrie_imu_test_pkg.xacro"/>
 </robot>

File: model/robots/valkyrie_sim.xacro (robot description, xacro)
@@ -11,5 +11,5 @@
     <xacro:include filename="$(find val_description)/model/urdf/multisense_sl.urdf" />
     <xacro:include filename="$(find val_description)/common/xacro/serial_numbers/valkyrie_A_serials.xacro"/>
-    <xacro:include filename="$(find val_description)/common/xacro/config_packages/valkyrie_A_pkg.xacro"/>
+    <xacro:include filename="$(find val_description)/common/xacro/config_packages/valkyrie_gazebo_pkg.xacro"/>
     <xacro:include filename="$(find val_description)/common/xacro/dev_ports/valkyrie_gazebo_ports.xacro"/>
     <xacro:include filename="$(find val_description)/model/robots/common/xacro/valkyrie_base_sim.xacro"/>

File: model/robots/valkyrie_sim_arm_mass_sims.xacro (robot description, xacro)
@@ -11,5 +11,5 @@
     <xacro:include filename="$(find val_description)/model/urdf/multisense_sl.urdf" />
     <xacro:include filename="$(find val_description)/common/xacro/serial_numbers/valkyrie_A_serials.xacro"/>
-    <xacro:include filename="$(find val_description)/common/xacro/config_packages/valkyrie_A_pkg.xacro"/>
+    <xacro:include filename="$(find val_description)/common/xacro/config_packages/valkyrie_gazebo_pkg.xacro"/>
     <xacro:include filename="$(find val_description)/common/xacro/dev_ports/valkyrie_gazebo_ports.xacro"/>
     <xacro:include filename="$(find val_description)/model/robots/common/xacro/valkyrie_arm_mass_sims_base_sim.xacro"/>

File: model/robots/valkyrie_sim_gazebo_sync.xacro (robot description, xacro)
@@ -12,5 +12,5 @@
     <xacro:include filename="$(find val_description)/model/urdf/multisense_sl.urdf" />
     <xacro:include filename="$(find val_description)/common/xacro/serial_numbers/valkyrie_A_serials.xacro"/>
-    <xacro:include filename="$(find val_description)/common/xacro/config_packages/valkyrie_A_pkg.xacro"/>
+    <xacro:include filename="$(find val_description)/common/xacro/config_packages/valkyrie_gazebo_pkg.xacro"/>
     <xacro:include filename="$(find val_description)/common/xacro/dev_ports/valkyrie_gazebo_ports.xacro"/>
     <xacro:include filename="$(find val_description)/model/robots/common/xacro/valkyrie_base_sim.xacro"/>

Commit message: updating for push to take a break from imu calibration

File: common/xacro/config_packages/valkyrie_A_pkg.xacro (robot description, xacro)
@@ -7,5 +7,5 @@
 	<xacro:property name="pelvis_rear_imu_pkg" value="val_config_files" />
 	<xacro:property name="torso_left_imu_pkg" value="val_config_files" />
-	<xacro:property name="pelvis_middle_imu_cal" value="None" />
+	<xacro:property name="pelvis_middle_imu_cal" value="3dm_gx4_15/47095/Calibration.cal" />
 	<xacro:property name="pelvis_rear_imu_cal" value="kvh_1750/1608K048/Calibration.cal" />
 	<xacro:property name="torso_left_imu_cal" value="3dm_gx4_15/47090/Calibration.cal" />

File: model/robots/common/xacro/valkyrie_base_hw.xacro (robot description, xacro)
@@ -23,5 +23,5 @@
     <xacro:v1_leg_sensors prefix="right" reflect="-1" ATI_node="${right_foot_ATI_node}" ATI_sensor_pkg="${right_foot_ATI_pkg}" ATI_config_file="${right_foot_ATI_cal}"/>
     <xacro:include_multisense_hw />
-    <xacro:v1_pelvis_rear_sensors_usb sensor_node_tag="${pelvis_rear_imu_node}" sensor_api_tag="${rearPelvisImuApi}"  sensor_pkg_tag="${pelvis_rear_imu_pkg}" sensor_config_tag="${pelvis_rear_imu_cal}" />
+    <xacro:v1_pelvis_sensors_usb middle_sensor_node_tag="${pelvis_middle_imu_node}" middle_sensor_api_tag="${middlePelvisImuApi}" middle_sensor_pkg_tag="${pelvis_middle_imu_pkg}" middle_sensor_config_tag="${pelvis_middle_imu_cal}" rear_sensor_node_tag="${pelvis_rear_imu_node}" rear_sensor_api_tag="${rearPelvisImuApi}" rear_sensor_pkg_tag="${pelvis_rear_imu_pkg}" rear_sensor_config_tag="${pelvis_rear_imu_cal}"/>
     <xacro:waist_transmissions_hw />
     <xacro:leg_transmissions_hw prefix="left"/>

Commit message: correcting xml error

File: common/xacro/config_packages/valkyrie_A_pkg.xacro (robot description, xacro)
@@ -8,5 +8,5 @@
 	<xacro:property name="torso_left_imu_pkg" value="val_config_files" />
 	<xacro:property name="pelvis_middle_imu_cal" value="3dm_gx4_15/47095/Calibration.cal" />
-	<xacro:property name="pelvis_rear_imu_cal" value="stim300/N25581710875719/Calibration.cal"
+	<xacro:property name="pelvis_rear_imu_cal" value="stim300/N25581710875719/Calibration.cal"/>
 	<xacro:property name="torso_left_imu_cal" value="3dm_gx4_15/47090/Calibration.cal" />
 </robot>
