Commit message: added imu to instance file and changed force torque sensor names to be consistant with urdf

File: common/xacro/api/valkyrie_A_api.xacro (robot description, xacro)
@@ -23,4 +23,5 @@
     <xacro:property name="ImuVectorNavHardwareApi" value="val_imu_vectornav_vn100_interface/ImuVecotNavInterface" />
     <xacro:property name="ImuSensorSimApi" value="val_imu_gazebo_interface/ImuGazeboInterface" />
+    <xacro:property name="ImuMicrostrainCalApi" value="imu_3dm_gx4_calibration/Imu3dmGx4Calibration"/>
     <xacro:property name="ThumbFingerApi" value="midas_finger_interface/MidasFingerAPI" />
     <xacro:property name="IndexFingerApi" value="midas_finger_interface/MidasFingerAPI"/>

File: common/xacro/api/valkyrie_B_api.xacro (robot description, xacro)
@@ -23,4 +23,5 @@
     <xacro:property name="ImuVectorNavHardwareApi" value="val_imu_vectornav_vn100_interface/ImuVecotNavInterface" />
     <xacro:property name="ImuSensorSimApi" value="val_imu_gazebo_interface/ImuGazeboInterface" />
+    <xacro:property name="ImuMicrostrainCalApi" value="imu_3dm_gx4_calibration/Imu3dmGx4Calibration"/>
     <xacro:property name="ThumbFingerApi" value="midas_finger_interface/MidasFingerAPI" />
     <xacro:property name="IndexFingerApi" value="midas_finger_interface/MidasFingerAPI"/>

File: common/xacro/api/valkyrie_C_api.xacro (robot description, xacro)
@@ -23,4 +23,5 @@
     <xacro:property name="ImuVectorNavHardwareApi" value="val_imu_vectornav_vn100_interface/ImuVecotNavInterface" />
     <xacro:property name="ImuSensorSimApi" value="val_imu_gazebo_interface/ImuGazeboInterface" />
+    <xacro:property name="ImuMicrostrainCalApi" value="imu_3dm_gx4_calibration/Imu3dmGx4Calibration"/>
     <xacro:property name="ThumbFingerApi" value="midas_finger_interface/MidasFingerAPI" />
     <xacro:property name="IndexFingerApi" value="midas_finger_interface/MidasFingerAPI"/>

File: instance/instances/robots/valkyrie_A.xacro (robot description, xacro)
@@ -2,4 +2,6 @@
 	<xacro:property name="instance" value="valkyrie_A" />
 	<xacro:include filename="$(find val_description)/common/xacro/serial_numbers/valkyrie_A_serials.xacro" />
+	<xacro:include filename="$(find val_description)/common/xacro/dev_ports/valkyrie_A_ports.xacro" />
+	<xacro:include filename="$(find val_description)/common/xacro/api/valkyrie_A_api.xacro" />
     <xacro:include filename="$(find val_description)/instance/instances/robots/xacro/common/valkyrie_full_template.xacro"/>
 </robot>

File: instance/instances/robots/valkyrie_B.xacro (robot description, xacro)
@@ -2,4 +2,6 @@
 	<xacro:property name="instance" value="valkyrie_B" />
 	<xacro:include filename="$(find val_description)/common/xacro/serial_numbers/valkyrie_B_serials.xacro" />
+	<xacro:include filename="$(find val_description)/common/xacro/dev_ports/valkyrie_B_ports.xacro" />
+	<xacro:include filename="$(find val_description)/common/xacro/api/valkyrie_B_api.xacro" />
     <xacro:include filename="$(find val_description)/instance/instances/robots/xacro/common/valkyrie_full_template.xacro"/>
 </robot>

File: instance/instances/robots/valkyrie_C.xacro (robot description, xacro)
@@ -2,4 +2,6 @@
 	<xacro:property name="instance" value="valkyrie_C" />
 	<xacro:include filename="$(find val_description)/common/xacro/serial_numbers/valkyrie_C_serials.xacro" />
+	<xacro:include filename="$(find val_description)/common/xacro/dev_ports/valkyrie_C_ports.xacro" />
+	<xacro:include filename="$(find val_description)/common/xacro/api/valkyrie_C_api.xacro" />
     <xacro:include filename="$(find val_description)/instance/instances/robots/xacro/common/valkyrie_full_template.xacro"/>
 </robot>

File: instance/instances/robots/valkyrie_D.xacro (robot description, xacro)
@@ -2,4 +2,6 @@
     <xacro:property name="instance" value="valkyrie_D" />
     <xacro:include filename="$(find val_description)/common/xacro/serial_numbers/valkyrie_D_serials.xacro" />
+    <xacro:include filename="$(find val_description)/common/xacro/dev_ports/valkyrie_D_ports.xacro" />
+    <xacro:include filename="$(find val_description)/common/xacro/api/valkyrie_D_api.xacro" />
     <xacro:include filename="$(find val_description)/instance/instances/robots/xacro/common/valkyrie_full_template.xacro"/>
 </robot>

File: instance/instances/robots/xacro/common/valkyrie_full_template.xacro (robot description, xacro)
@@ -19,6 +19,8 @@
 	</Mechanisms>
 	<Devices>
-		<xacro:ati_force_torque name="left_foot_force_torque" serial_number="${left_foot_ATI_serial}" node="${left_foot_ATI_node}"/>
-		<xacro:ati_force_torque name="right_foot_force_torque" serial_number="${right_foot_ATI_serial}" node="${right_foot_ATI_node}"/>
+		<xacro:ati_force_torque name="leftFootSixAxis" serial_number="${left_foot_ATI_serial}" node="${left_foot_ATI_node}"/>
+		<xacro:ati_force_torque name="rightFootSixAxis" serial_number="${right_foot_ATI_serial}" node="${right_foot_ATI_node}"/>
+		<xacro:imu_device name="pelvisRearImu" DevicePort="${pelvis_rear_imu_port}" DeviceAPI="${ImuMicrostrainCalApi}"/>
+		<xacro:imu_device name="torsoLeftImu" DevicePort="${torso_left_imu_port}" DeviceAPI="${ImuMicrostrainCalApi}" />
 	</Devices>
 </robot>

File: instance/instances/robots/xacro/sensors/imu.xacro (robot description, xacro)
@@ -1,7 +1,7 @@
 <robot xmlns:xacro="http://ros.org/wiki/xacro" name="imu">
-	<xacro:macro name="microstrain_imu" params="name serial_number node">
+	<xacro:macro name="imu_device" params="name DevicePort DeviceAPI">
 		<Device id="${name}" type="imu">
-			<SerialNumber id="${serial_number}" />
-			<Node id="${node}" />
+			<DevicePort id="${DevicePort}" />
+			<DeviceAPI id="${DeviceAPI}" />
 		</Device>
 	</xacro:macro>

Commit message: added versitility to imu api creation for urdf

File: common/xacro/api/valkyrie_A_api.xacro (robot description, xacro)
@@ -21,6 +21,10 @@
     <xacro:property name="ForceTorqueSensorApi" value="ati_sensor_interface::ATISensorInterface" />
     <xacro:property name="ImuMicrostrainHardwareApi" value="imu_3dm_gx4_15_sensor::Imu3DmGx415Sensor" />
+    <xacro:property name="ImuKVHHardwareApi" value="kvh_1750_sensor::KVH1750ConstSensor" />
     <xacro:property name="ImuVectorNavHardwareApi" value="val_imu_vectornav_vn100_interface/ImuVecotNavInterface" />
     <xacro:property name="ImuSensorSimApi" value="val_imu_gazebo_interface/ImuGazeboInterface" />
+    <xacro:property name="rearPelvisImuApi" value="${ImuKVHHardwareApi}" />
+    <xacro:property name="middlePelvisImuApi" value="${ImuMicrostrainHardwareApi}" />
+    <xacro:property name="trunkImuApi" value="${ImuMicrostrainHardwareApi}" />
     <xacro:property name="ThumbFingerApi" value="midas_finger_interface/MidasFingerAPI" />
     <xacro:property name="IndexFingerApi" value="midas_finger_interface/MidasFingerAPI"/>

File: common/xacro/api/valkyrie_B_api.xacro (robot description, xacro)
@@ -21,6 +21,10 @@
     <xacro:property name="ForceTorqueSensorApi" value="ati_sensor_interface::ATISensorInterface" />
     <xacro:property name="ImuMicrostrainHardwareApi" value="imu_3dm_gx4_15_sensor::Imu3DmGx415Sensor" />
+    <xacro:property name="ImuKVHHardwareApi" value="kvh_1750_sensor::KVH1750ConstSensor" />
     <xacro:property name="ImuVectorNavHardwareApi" value="val_imu_vectornav_vn100_interface/ImuVecotNavInterface" />
     <xacro:property name="ImuSensorSimApi" value="val_imu_gazebo_interface/ImuGazeboInterface" />
+    <xacro:property name="rearPelvisImuApi" value="${ImuMicrostrainHardwareApi}" />
+    <xacro:property name="middlePelvisImuApi" value="${ImuMicrostrainHardwareApi}" />
+    <xacro:property name="trunkImuApi" value="${ImuMicrostrainHardwareApi}" />
     <xacro:property name="ThumbFingerApi" value="midas_finger_interface/MidasFingerAPI" />
     <xacro:property name="IndexFingerApi" value="midas_finger_interface/MidasFingerAPI"/>

File: common/xacro/api/valkyrie_C_api.xacro (robot description, xacro)
@@ -21,6 +21,10 @@
     <xacro:property name="ForceTorqueSensorApi" value="ati_sensor_interface::ATISensorInterface" />
     <xacro:property name="ImuMicrostrainHardwareApi" value="imu_3dm_gx4_15_sensor::Imu3DmGx415Sensor" />
+    <xacro:property name="ImuKVHHardwareApi" value="kvh_1750_sensor::KVH1750ConstSensor" />
     <xacro:property name="ImuVectorNavHardwareApi" value="val_imu_vectornav_vn100_interface/ImuVecotNavInterface" />
     <xacro:property name="ImuSensorSimApi" value="val_imu_gazebo_interface/ImuGazeboInterface" />
+    <xacro:property name="rearPelvisImuApi" value="${ImuMicrostrainHardwareApi}" />
+    <xacro:property name="middlePelvisImuApi" value="${ImuMicrostrainHardwareApi}" />
+    <xacro:property name="trunkImuApi" value="${ImuMicrostrainHardwareApi}" />
     <xacro:property name="ThumbFingerApi" value="midas_finger_interface/MidasFingerAPI" />
     <xacro:property name="IndexFingerApi" value="midas_finger_interface/MidasFingerAPI"/>

File: common/xacro/api/valkyrie_sim_api.xacro (robot description, xacro)
@@ -3,3 +3,6 @@
     <xacro:property name="ImuSensorSimApi" value="simulated_imu_sensor::SimulatedImuSensor" />
     <xacro:property name="ForceTorqueSensorApi" value="sensor_interface::SimForceTorqueSensor" />
+    <xacro:property name="rearPelvisImuApi" value="${ImuSensorSimApi}" />
+    <xacro:property name="middlePelvisImuApi" value="${ImuSensorSimApi}" />
+    <xacro:property name="trunkImuApi" value="${ImuSensorSimApi}" />
 </robot>

File: common/xacro/config_packages/valkyrie_A_pkg.xacro (robot description, xacro)
@@ -8,5 +8,5 @@
 	<xacro:property name="torso_left_imu_pkg" value="val_config_files" />
 	<xacro:property name="pelvis_middle_imu_cal" value="None" />
-	<xacro:property name="pelvis_rear_imu_cal" value="3dm_gx4_15/47090/Calibration.cal" />
-	<xacro:property name="torso_left_imu_cal" value="3dm_gx4_15/47095/Calibration.cal" />
+	<xacro:property name="pelvis_rear_imu_cal" value="kvh_1750/1608K048/Calibration.cal" />
+	<xacro:property name="torso_left_imu_cal" value="3dm_gx4_15/47090/Calibration.cal" />
 </robot>

File: model/robots/common/xacro/valkyrie_arm_mass_sims_base_hw.xacro (robot description, xacro)
@@ -11,9 +11,9 @@
     <xacro:make_leg prefix="right" reflect="-1" leg_root_link="${Pelvis_Link_Name}"/>
     <xacro:make_leg prefix="left" reflect="1" leg_root_link="${Pelvis_Link_Name}"/>
-    <xacro:v1_trunk_sensors_usb sensor_node_tag="${torso_left_imu_node}" sensor_api_tag="${ImuMicrostrainHardwareApi}" sensor_pkg_tag="${torso_left_imu_pkg}" sensor_config_tag="${torso_left_imu_cal}" />
+    <xacro:v1_trunk_sensors_usb sensor_node_tag="${torso_left_imu_node}" sensor_api_tag="${trunkImuApi}" sensor_pkg_tag="${torso_left_imu_pkg}" sensor_config_tag="${torso_left_imu_cal}" />
     <xacro:v1_leg_sensors prefix="left" reflect="1" ATI_node="${left_foot_ATI_node}" ATI_sensor_pkg="${left_foot_ATI_pkg}" ATI_config_file="${left_foot_ATI_cal}"/>
     <xacro:v1_leg_sensors prefix="right" reflect="-1" ATI_node="${right_foot_ATI_node}" ATI_sensor_pkg="${right_foot_ATI_pkg}" ATI_config_file="${right_foot_ATI_cal}"/>
     <xacro:include_multisense_hw />
-    <xacro:v1_pelvis_rear_sensors_usb sensor_node_tag="${pelvis_rear_imu_node}" sensor_api_tag="${ImuMicrostrainHardwareApi}"  sensor_pkg_tag="${pelvis_rear_imu_pkg}" sensor_config_tag="${pelvis_rear_imu_cal}" />
+    <xacro:v1_pelvis_rear_sensors_usb sensor_node_tag="${pelvis_rear_imu_node}" sensor_api_tag="${rearPelvisImuApi}"  sensor_pkg_tag="${pelvis_rear_imu_pkg}" sensor_config_tag="${pelvis_rear_imu_cal}" />
     <xacro:waist_transmissions_hw />
     <xacro:leg_transmissions_hw prefix="left"/>

File: model/robots/common/xacro/valkyrie_arm_mass_sims_base_sim.xacro (robot description, xacro)
@@ -11,9 +11,9 @@
     <xacro:make_leg prefix="right" reflect="-1" leg_root_link="${Pelvis_Link_Name}"/>
     <xacro:make_leg prefix="left" reflect="1" leg_root_link="${Pelvis_Link_Name}"/>
-    <xacro:v1_pelvis_sensors_usb middle_sensor_node_tag="${pelvis_middle_imu_node}" middle_sensor_api_tag="${ImuSensorSimApi}" middle_sensor_pkg_tag="${pelvis_middle_imu_pkg}" middle_sensor_config_tag="${pelvis_middle_imu_cal}" rear_sensor_node_tag="${pelvis_rear_imu_node}" rear_sensor_api_tag="${ImuSensorSimApi}" rear_sensor_pkg_tag="${pelvis_rear_imu_pkg}" rear_sensor_config_tag="${pelvis_rear_imu_cal}"/>
+    <xacro:v1_pelvis_sensors_usb middle_sensor_node_tag="${pelvis_middle_imu_node}" middle_sensor_api_tag="${middlePelvisImuApi}" middle_sensor_pkg_tag="${pelvis_middle_imu_pkg}" middle_sensor_config_tag="${pelvis_middle_imu_cal}" rear_sensor_node_tag="${pelvis_rear_imu_node}" rear_sensor_api_tag="${rearPelvisImuApi}" rear_sensor_pkg_tag="${pelvis_rear_imu_pkg}" rear_sensor_config_tag="${pelvis_rear_imu_cal}"/>
     <xacro:v1_leg_sensors prefix="left" reflect="1" ATI_node="${left_foot_ATI_node}" ATI_sensor_pkg="${left_foot_ATI_pkg}" ATI_config_file="${left_foot_ATI_cal}"/>
     <xacro:v1_leg_sensors prefix="right" reflect="-1" ATI_node="${right_foot_ATI_node}" ATI_sensor_pkg="${right_foot_ATI_pkg}" ATI_config_file="${right_foot_ATI_cal}"/>
     <xacro:include_multisense_sim />
-    <xacro:v1_trunk_sensors_usb sensor_node_tag="${torso_left_imu_node}" sensor_api_tag="${ImuSensorSimApi}" sensor_pkg_tag="${torso_left_imu_pkg}" sensor_config_tag="${torso_left_imu_cal}" />
+    <xacro:v1_trunk_sensors_usb sensor_node_tag="${torso_left_imu_node}" sensor_api_tag="${trunkImuApi}" sensor_pkg_tag="${torso_left_imu_pkg}" sensor_config_tag="${torso_left_imu_cal}" />
     <xacro:waist_transmissions_sim />
     <xacro:leg_transmissions_sim prefix="left"/>

File: model/robots/common/xacro/valkyrie_base_hw.xacro (robot description, xacro)
@@ -19,9 +19,9 @@
     <xacro:make_leg prefix="right" reflect="-1" leg_root_link="${Pelvis_Link_Name}"/>
     <xacro:make_leg prefix="left" reflect="1" leg_root_link="${Pelvis_Link_Name}"/>
-    <xacro:v1_trunk_sensors_usb sensor_node_tag="${torso_left_imu_node}" sensor_api_tag="${ImuMicrostrainHardwareApi}" sensor_pkg_tag="${torso_left_imu_pkg}" sensor_config_tag="${torso_left_imu_cal}" />
+    <xacro:v1_trunk_sensors_usb sensor_node_tag="${torso_left_imu_node}" sensor_api_tag="${trunkImuApi}" sensor_pkg_tag="${torso_left_imu_pkg}" sensor_config_tag="${torso_left_imu_cal}" />
     <xacro:v1_leg_sensors prefix="left" reflect="1" ATI_node="${left_foot_ATI_node}" ATI_sensor_pkg="${left_foot_ATI_pkg}" ATI_config_file="${left_foot_ATI_cal}"/>
     <xacro:v1_leg_sensors prefix="right" reflect="-1" ATI_node="${right_foot_ATI_node}" ATI_sensor_pkg="${right_foot_ATI_pkg}" ATI_config_file="${right_foot_ATI_cal}"/>
     <xacro:include_multisense_hw />
-    <xacro:v1_pelvis_rear_sensors_usb sensor_node_tag="${pelvis_rear_imu_node}" sensor_api_tag="${ImuMicrostrainHardwareApi}"  sensor_pkg_tag="${pelvis_rear_imu_pkg}" sensor_config_tag="${pelvis_rear_imu_cal}" />
+    <xacro:v1_pelvis_rear_sensors_usb sensor_node_tag="${pelvis_rear_imu_node}" sensor_api_tag="${rearPelvisImuApi}"  sensor_pkg_tag="${pelvis_rear_imu_pkg}" sensor_config_tag="${pelvis_rear_imu_cal}" />
     <xacro:waist_transmissions_hw />
     <xacro:leg_transmissions_hw prefix="left"/>

File: model/robots/common/xacro/valkyrie_base_sim.xacro (robot description, xacro)
@@ -19,9 +19,9 @@
     <xacro:make_leg prefix="right" reflect="-1" leg_root_link="${Pelvis_Link_Name}"/>
     <xacro:make_leg prefix="left" reflect="1" leg_root_link="${Pelvis_Link_Name}"/>
-    <xacro:v1_pelvis_sensors_usb middle_sensor_node_tag="${pelvis_middle_imu_node}" middle_sensor_api_tag="${ImuSensorSimApi}" middle_sensor_pkg_tag="${pelvis_middle_imu_pkg}" middle_sensor_config_tag="${pelvis_middle_imu_cal}" rear_sensor_node_tag="${pelvis_rear_imu_node}" rear_sensor_api_tag="${ImuSensorSimApi}" rear_sensor_pkg_tag="${pelvis_rear_imu_pkg}" rear_sensor_config_tag="${pelvis_rear_imu_cal}"/>
+    <xacro:v1_pelvis_sensors_usb middle_sensor_node_tag="${pelvis_middle_imu_node}" middle_sensor_api_tag="${middlePelvisImuApi}" middle_sensor_pkg_tag="${pelvis_middle_imu_pkg}" middle_sensor_config_tag="${pelvis_middle_imu_cal}" rear_sensor_node_tag="${pelvis_rear_imu_node}" rear_sensor_api_tag="${rearPelvisImuApi}" rear_sensor_pkg_tag="${pelvis_rear_imu_pkg}" rear_sensor_config_tag="${pelvis_rear_imu_cal}"/>
     <xacro:v1_leg_sensors prefix="left" reflect="1" ATI_node="${left_foot_ATI_node}" ATI_sensor_pkg="${left_foot_ATI_pkg}" ATI_config_file="${left_foot_ATI_cal}"/>
     <xacro:v1_leg_sensors prefix="right" reflect="-1" ATI_node="${right_foot_ATI_node}" ATI_sensor_pkg="${right_foot_ATI_pkg}" ATI_config_file="${right_foot_ATI_cal}"/>
     <xacro:include_multisense_sim />
-    <xacro:v1_trunk_sensors_usb sensor_node_tag="${torso_left_imu_node}" sensor_api_tag="${ImuSensorSimApi}" sensor_pkg_tag="${torso_left_imu_pkg}" sensor_config_tag="${torso_left_imu_cal}" />
+    <xacro:v1_trunk_sensors_usb sensor_node_tag="${torso_left_imu_node}" sensor_api_tag="${trunkImuApi}" sensor_pkg_tag="${torso_left_imu_pkg}" sensor_config_tag="${torso_left_imu_cal}" />
     <xacro:waist_transmissions_sim />
     <xacro:leg_transmissions_sim prefix="left"/>

Commit message: moving kvh imu to separate feature branch

File: common/xacro/api/valkyrie_A_api.xacro (robot description, xacro)
@@ -21,6 +21,5 @@
     <xacro:property name="ForceTorqueSensorApi" value="ati_sensor_interface::ATISensorInterface" />
     <xacro:property name="ImuMicrostrainHardwareApi" value="imu_3dm_gx4_15_sensor::Imu3DmGx415Sensor" />
-    <xacro:property name="ImuKVHHardwareApi" value="kvh_1750_sensor::KVH1750ConstSensor" />
-    <xacro:property name="ImuVectorNavHardwareApi" value="val_imu_vectornav_vn100_interface/ImuVecotNavInterface" />
+    <xacro:property name="ImuStimHardwareApi" value="stim_300_sensor::STIM300ConstSensor" />
     <xacro:property name="ImuSensorSimApi" value="val_imu_gazebo_interface/ImuGazeboInterface" />
     <xacro:property name="rearPelvisImuApi" value="${ImuKVHHardwareApi}" />

File: common/xacro/config_packages/valkyrie_A_pkg.xacro (robot description, xacro)
@@ -8,5 +8,5 @@
 	<xacro:property name="torso_left_imu_pkg" value="val_config_files" />
 	<xacro:property name="pelvis_middle_imu_cal" value="3dm_gx4_15/47095/Calibration.cal" />
-	<xacro:property name="pelvis_rear_imu_cal" value="kvh_1750/1608K048/Calibration.cal" />
+	<xacro:property name="pelvis_rear_imu_cal" value="stim300/N25581710875719/Calibration.cal"
 	<xacro:property name="torso_left_imu_cal" value="3dm_gx4_15/47090/Calibration.cal" />
 </robot>

File: model/robots/common/xacro/valkyrie_imu_base.xacro (robot description, xacro)
@@ -1,4 +1,3 @@
 <robot xmlns:xacro="http://ros.org/wiki/xacro" name="valkyrie_imu_base">
-    <xacro:property name="KVHHardwareApi" value="kvh_1750_sensor::KVH1750ConstSensor" />
     <xacro:property name="MicroStrainHardwareApi" value="imu_3dm_gx4_15_sensor::Imu3DmGx415Sensor" />
     <xacro:property name="StimHardwareApi" value="stim_300_sensor::STIM300ConstSensor" />

Commit message: removing more kvh tags

File: common/xacro/api/valkyrie_A_api.xacro (robot description, xacro)
@@ -23,5 +23,5 @@
     <xacro:property name="ImuStimHardwareApi" value="stim_300_sensor::STIM300ConstSensor" />
     <xacro:property name="ImuSensorSimApi" value="val_imu_gazebo_interface/ImuGazeboInterface" />
-    <xacro:property name="rearPelvisImuApi" value="${ImuKVHHardwareApi}" />
+    <xacro:property name="rearPelvisImuApi" value="${ImuStimHardwareApi}" />
     <xacro:property name="middlePelvisImuApi" value="${ImuMicrostrainHardwareApi}" />
     <xacro:property name="trunkImuApi" value="${ImuMicrostrainHardwareApi}" />

File: common/xacro/api/valkyrie_B_api.xacro (robot description, xacro)
@@ -21,6 +21,5 @@
     <xacro:property name="ForceTorqueSensorApi" value="ati_sensor_interface::ATISensorInterface" />
     <xacro:property name="ImuMicrostrainHardwareApi" value="imu_3dm_gx4_15_sensor::Imu3DmGx415Sensor" />
-    <xacro:property name="ImuKVHHardwareApi" value="kvh_1750_sensor::KVH1750ConstSensor" />
-    <xacro:property name="ImuVectorNavHardwareApi" value="val_imu_vectornav_vn100_interface/ImuVecotNavInterface" />
+    <xacro:property name="ImuStimHardwareApi" value="stim_300_sensor::STIM300ConstSensor" />
     <xacro:property name="ImuSensorSimApi" value="val_imu_gazebo_interface/ImuGazeboInterface" />
     <xacro:property name="rearPelvisImuApi" value="${ImuMicrostrainHardwareApi}" />

File: common/xacro/api/valkyrie_C_api.xacro (robot description, xacro)
@@ -21,6 +21,5 @@
     <xacro:property name="ForceTorqueSensorApi" value="ati_sensor_interface::ATISensorInterface" />
     <xacro:property name="ImuMicrostrainHardwareApi" value="imu_3dm_gx4_15_sensor::Imu3DmGx415Sensor" />
-    <xacro:property name="ImuKVHHardwareApi" value="kvh_1750_sensor::KVH1750ConstSensor" />
-    <xacro:property name="ImuVectorNavHardwareApi" value="val_imu_vectornav_vn100_interface/ImuVecotNavInterface" />
+    <xacro:property name="ImuStimHardwareApi" value="stim_300_sensor::STIM300ConstSensor" />
     <xacro:property name="ImuSensorSimApi" value="val_imu_gazebo_interface/ImuGazeboInterface" />
     <xacro:property name="rearPelvisImuApi" value="${ImuMicrostrainHardwareApi}" />

File: common/xacro/config_packages/valkyrie_imu_test_pkg.xacro (robot description, xacro)
@@ -3,5 +3,4 @@
 	<xacro:property name="pelvis_rear_imu_pkg" value="val_config_files" />
 	<xacro:property name="pelvis_test_imu_pkg" value="val_config_files" />
-	<xacro:property name="pelvis_middle_imu_cal" value="kvh_1750/1608K048/Calibration.cal" />
 	<xacro:property name="pelvis_rear_imu_cal" value="3dm_gx4_15/47099/Calibration.cal" />
 	<xacro:property name="pelvis_test_imu_cal" value="stim300/N25581710875719/Calibration.cal" />
