Commit message: correcting issue with xacro tags

File: model/robots/common/xacro/pelvis/pelvis.xacro (robot description, xacro)
@@ -66,4 +66,4 @@
                                   sensor_pkg="${middle_sensor_pkg_tag}"
                                   sensor_config_file="${middle_sensor_config_tag}" />
-    </xacro:macro
+    </xacro:macro>
 </robot>

File: model/robots/common/xacro/waist/angled_j1s_includes.xacro (robot description, xacro)
@@ -9,5 +9,5 @@
   <xacro:include filename="$(find val_description)/common/xacro/joint_names/valkyrie_joint_names.xacro"/>
   <xacro:include filename="$(find val_description)/common/xacro/actuator_names/valkyrie_actuator_names.xacro"/>
-  <xacro:include filename="$(find val_description)/model/robots/common/xacro/sensors/microstrain.xacro"/>
+  <xacro:include filename="$(find val_description)/model/robots/common/xacro/sensors/inertial_measurement_unit.xacro"/>
   <xacro:include filename="$(find val_description)/model/robots/common/xacro/sensors/flea.xacro"/>
   <xacro:include filename="$(find val_description)/model/robots/common/xacro/waist/waist.xacro"/>

File: model/robots/common/xacro/waist/waist.xacro (robot description, xacro)
@@ -1,13 +1,3 @@
 <robot xmlns:xacro="http://www.ros.org/wiki/xacro" name="waist">
-  <xacro:include filename="$(find val_description)/common/xacro/joint_names/valkyrie_joint_names.xacro"/>
-  <xacro:include filename="$(find val_description)/common/xacro/actuator_names/valkyrie_actuator_names.xacro"/>
-  <xacro:include filename="$(find val_description)/model/robots/common/xacro/waist/joint_axes.xacro"/>
-  <xacro:include filename="$(find val_description)/model/robots/common/xacro/waist/joint_axes.xacro"/>
-  <xacro:include filename="$(find val_description)/model/robots/common/xacro/waist/link_names.xacro"/>
-  <xacro:include filename="$(find val_description)/model/robots/common/xacro/waist/joint_limits.xacro"/>
-  <xacro:include filename="$(find val_description)/model/robots/common/xacro/waist/frame_parameters.xacro"/>
-  <xacro:include filename="$(find val_description)/model/robots/common/xacro/waist/mass_parameters.xacro"/>
-  <xacro:include filename="$(find val_description)/model/robots/common/xacro/sensors/inertial_measurement_unit.xacro"/>
-  <xacro:include filename="$(find val_description)/model/robots/common/xacro/sensors/flea.xacro"/>
   <xacro:macro name="make_waist_common" params="waist_root_link">
     <xacro:revolute_joint_ex jointName="${TorsoYawJointName}"

File: model/robots/common/xacro/waist/waist_includes.xacro (robot description, xacro)
@@ -1,13 +1,13 @@
 <robot xmlns:xacro="http://ros.org/wiki/xacro" name="waist_includes">
-	<xacro:include filename="$(find val_description)/model/robots/common/xacro/waist/joint_axes.xacro"/>
-	<xacro:include filename="$(find val_description)/model/robots/common/xacro/waist/joint_axes.xacro"/>
-	<xacro:include filename="$(find val_description)/model/robots/common/xacro/waist/link_names.xacro"/>
-	<xacro:include filename="$(find val_description)/model/robots/common/xacro/waist/joint_limits.xacro"/>
-	<xacro:include filename="$(find val_description)/model/robots/common/xacro/waist/frame_parameters.xacro"/>
-	<xacro:include filename="$(find val_description)/model/robots/common/xacro/waist/mass_parameters.xacro"/>
-	<xacro:include filename="$(find val_description)/common/xacro/joint_names/valkyrie_joint_names.xacro"/>
-	<xacro:include filename="$(find val_description)/common/xacro/actuator_names/valkyrie_actuator_names.xacro"/>
-	<xacro:include filename="$(find val_description)/model/robots/common/xacro/sensors/microstrain.xacro"/>
-	<xacro:include filename="$(find val_description)/model/robots/common/xacro/sensors/flea.xacro"/>
+  <xacro:include filename="$(find val_description)/common/xacro/joint_names/valkyrie_joint_names.xacro"/>
+  <xacro:include filename="$(find val_description)/common/xacro/actuator_names/valkyrie_actuator_names.xacro"/>
+  <xacro:include filename="$(find val_description)/model/robots/common/xacro/waist/joint_axes.xacro"/>
+  <xacro:include filename="$(find val_description)/model/robots/common/xacro/waist/joint_axes.xacro"/>
+  <xacro:include filename="$(find val_description)/model/robots/common/xacro/waist/link_names.xacro"/>
+  <xacro:include filename="$(find val_description)/model/robots/common/xacro/waist/joint_limits.xacro"/>
+  <xacro:include filename="$(find val_description)/model/robots/common/xacro/waist/frame_parameters.xacro"/>
+  <xacro:include filename="$(find val_description)/model/robots/common/xacro/waist/mass_parameters.xacro"/>
+  <xacro:include filename="$(find val_description)/model/robots/common/xacro/sensors/inertial_measurement_unit.xacro"/>
+  <xacro:include filename="$(find val_description)/model/robots/common/xacro/sensors/flea.xacro"/>
 	<xacro:include filename="$(find val_description)/model/robots/common/xacro/waist/waist.xacro"/>
 </robot>

File: model/robots/valkyrie_A.xacro (robot description, xacro)
@@ -1,3 +1,4 @@
 <robot xmlns:xacro="http://ros.org/wiki/xacro" name="valkyrie">
+    <xacro:property name="mesh_root" value="package://val_description/model/meshes"/>
 	<xacro:property name="leg_mesh_dir" value="package://val_description/model/meshes/legs"/>
     <xacro:property name="arm_mesh_dir" value="package://val_description/model/meshes/arms"/>
@@ -13,5 +14,4 @@
     <xacro:include filename="$(find val_description)/common/xacro/api/valkyrie_A_api.xacro"/>
     <xacro:include filename="$(find val_description)/common/xacro/config_packages/valkyrie_A_pkg.xacro"/>
-    <xacro:include filename="$(find val_description)/common/xacro/dev_ports/valkyrie_A_ports.xacro"/>
     <xacro:include filename="$(find val_description)/model/robots/common/xacro/common_bodies.xacro" />
     <!-- Pelvis include -->

File: model/robots/valkyrie_A_arm_mass_sims.xacro (robot description, xacro)
@@ -1,3 +1,4 @@
 <robot xmlns:xacro="http://ros.org/wiki/xacro" name="valkyrie">
+    <xacro:property name="mesh_root" value="package://val_description/model/meshes"/>
 	<xacro:property name="leg_mesh_dir" value="package://val_description/model/meshes/legs"/>
     <xacro:property name="arm_mesh_dir" value="package://val_description/model/meshes/arms"/>
@@ -13,5 +14,4 @@
     <xacro:include filename="$(find val_description)/common/xacro/api/valkyrie_A_api.xacro"/>
     <xacro:include filename="$(find val_description)/common/xacro/config_packages/valkyrie_A_pkg.xacro"/>
-    <xacro:include filename="$(find val_description)/common/xacro/dev_ports/valkyrie_A_ports.xacro"/>
     <!-- Pelvis include -->
     <xacro:include filename="$(find val_description)/model/robots/common/xacro/pelvis/pelvis_includes.xacro"/>

File: model/robots/valkyrie_B.xacro (robot description, xacro)
@@ -1,3 +1,4 @@
 <robot xmlns:xacro="http://ros.org/wiki/xacro" name="valkyrie">
+    <xacro:property name="mesh_root" value="package://val_description/model/meshes"/>
 	<xacro:property name="leg_mesh_dir" value="package://val_description/model/meshes/legs"/>
     <xacro:property name="arm_mesh_dir" value="package://val_description/model/meshes/arms"/>
@@ -13,5 +14,4 @@
     <xacro:include filename="$(find val_description)/common/xacro/api/valkyrie_B_api.xacro"/>
     <xacro:include filename="$(find val_description)/common/xacro/config_packages/valkyrie_B_pkg.xacro"/>
-    <xacro:include filename="$(find val_description)/common/xacro/dev_ports/valkyrie_B_ports.xacro"/>
     <xacro:include filename="$(find val_description)/model/robots/common/xacro/common_bodies.xacro" />
     <!-- Pelvis include -->

File: model/robots/valkyrie_B_arm_mass_sims.xacro (robot description, xacro)
@@ -1,3 +1,4 @@
 <robot xmlns:xacro="http://ros.org/wiki/xacro" name="valkyrie">
+    <xacro:property name="mesh_root" value="package://val_description/model/meshes"/>
 	<xacro:property name="leg_mesh_dir" value="package://val_description/model/meshes/legs"/>
     <xacro:property name="arm_mesh_dir" value="package://val_description/model/meshes/arms"/>
@@ -13,5 +14,4 @@
     <xacro:include filename="$(find val_description)/common/xacro/api/valkyrie_B_api.xacro"/>
     <xacro:include filename="$(find val_description)/common/xacro/config_packages/valkyrie_B_pkg.xacro"/>
-    <xacro:include filename="$(find val_description)/common/xacro/dev_ports/valkyrie_B_ports.xacro"/>
     <!-- Pelvis include -->
     <xacro:include filename="$(find val_description)/model/robots/common/xacro/pelvis/pelvis_includes.xacro"/>

File: model/robots/valkyrie_C.xacro (robot description, xacro)
@@ -1,3 +1,4 @@
 <robot xmlns:xacro="http://ros.org/wiki/xacro" name="valkyrie">
+    <xacro:property name="mesh_root" value="package://val_description/model/meshes"/>
 	<xacro:property name="leg_mesh_dir" value="package://val_description/model/meshes/legs"/>
     <xacro:property name="arm_mesh_dir" value="package://val_description/model/meshes/arms"/>
@@ -13,5 +14,4 @@
     <xacro:include filename="$(find val_description)/common/xacro/api/valkyrie_C_api.xacro"/>
     <xacro:include filename="$(find val_description)/common/xacro/config_packages/valkyrie_C_pkg.xacro"/>
-    <xacro:include filename="$(find val_description)/common/xacro/dev_ports/valkyrie_C_ports.xacro"/>
     <xacro:include filename="$(find val_description)/model/robots/common/xacro/common_bodies.xacro" />
     <!-- Pelvis include -->

File: model/robots/valkyrie_C_arm_mass_sims.xacro (robot description, xacro)
@@ -1,3 +1,4 @@
 <robot xmlns:xacro="http://ros.org/wiki/xacro" name="valkyrie">
+    <xacro:property name="mesh_root" value="package://val_description/model/meshes"/>
 	<xacro:property name="leg_mesh_dir" value="package://val_description/model/meshes/legs"/>
     <xacro:property name="arm_mesh_dir" value="package://val_description/model/meshes/arms"/>
@@ -13,5 +14,4 @@
     <xacro:include filename="$(find val_description)/common/xacro/api/valkyrie_C_api.xacro"/>
     <xacro:include filename="$(find val_description)/common/xacro/config_packages/valkyrie_C_pkg.xacro"/>
-    <xacro:include filename="$(find val_description)/common/xacro/dev_ports/valkyrie_C_ports.xacro"/>
     <!-- Pelvis include -->
     <xacro:include filename="$(find val_description)/model/robots/common/xacro/pelvis/pelvis_includes.xacro"/>

File: model/robots/valkyrie_D.xacro (robot description, xacro)
@@ -1,4 +1,5 @@
 <robot xmlns:xacro="http://ros.org/wiki/xacro" name="valkyrie">
-	<xacro:property name="leg_mesh_dir" value="package://val_description/model/meshes/legs"/>
+	<xacro:property name="mesh_root" value="package://val_description/model/meshes"/>
+    <xacro:property name="leg_mesh_dir" value="package://val_description/model/meshes/legs"/>
     <xacro:property name="arm_mesh_dir" value="package://val_description/model/meshes/arms"/>
     <xacro:property name="waist_mesh_dir" value="package://val_description/model/meshes/torso"/>
@@ -13,5 +14,4 @@
     <xacro:include filename="$(find val_description)/common/xacro/api/valkyrie_D_api.xacro"/>
     <xacro:include filename="$(find val_description)/common/xacro/config_packages/valkyrie_D_pkg.xacro"/>
-    <xacro:include filename="$(find val_description)/common/xacro/dev_ports/valkyrie_D_ports.xacro"/>
     <xacro:include filename="$(find val_description)/model/robots/common/xacro/common_bodies.xacro" />
     <!-- Pelvis include -->

File: model/robots/valkyrie_D_arm_mass_sims.xacro (robot description, xacro)
@@ -1,4 +1,5 @@
 <robot xmlns:xacro="http://ros.org/wiki/xacro" name="valkyrie">
-	<xacro:property name="leg_mesh_dir" value="package://val_description/model/meshes/legs"/>
+	<xacro:property name="mesh_root" value="package://val_description/model/meshes"/>
+    <xacro:property name="leg_mesh_dir" value="package://val_description/model/meshes/legs"/>
     <xacro:property name="arm_mesh_dir" value="package://val_description/model/meshes/arms"/>
     <xacro:property name="waist_mesh_dir" value="package://val_description/model/meshes/torso"/>
@@ -13,5 +14,4 @@
     <xacro:include filename="$(find val_description)/common/xacro/api/valkyrie_D_api.xacro"/>
     <xacro:include filename="$(find val_description)/common/xacro/config_packages/valkyrie_D_pkg.xacro"/>
-    <xacro:include filename="$(find val_description)/common/xacro/dev_ports/valkyrie_D_ports.xacro"/>
     <!-- Pelvis include -->
     <xacro:include filename="$(find val_description)/model/robots/common/xacro/pelvis/pelvis_includes.xacro"/>

File: model/robots/valkyrie_sim.xacro (robot description, xacro)
@@ -1,3 +1,4 @@
 <robot xmlns:xacro="http://ros.org/wiki/xacro" name="valkyrie">
+    <xacro:property name="mesh_root" value="package://val_description/model/meshes"/>
     <gazebo>
       <plugin filename="libval_gazebo.so" name="SharedMemorySimInterfacePlugin">

File: model/robots/valkyrie_sim_angled_legj1s.xacro (robot description, xacro)
@@ -1,3 +1,4 @@
 <robot xmlns:xacro="http://ros.org/wiki/xacro" name="valkyrie">
+    <xacro:property name="mesh_root" value="package://val_description/model/meshes"/>
     <gazebo>
       <plugin filename="libval_gazebo.so" name="SharedMemorySimInterfacePlugin">
@@ -18,5 +19,5 @@
     <xacro:include filename="$(find val_description)/model/urdf/multisense_sl.urdf" />
     <xacro:include filename="$(find val_description)/common/xacro/serial_numbers/valkyrie_A_serials.xacro"/>
-    <xacro:include filename="$(find val_description)/common/xacro/dev_ports/valkyrie_gazebo_ports.xacro"/>
+    <xacro:include filename="$(find val_description)/common/xacro/config_packages/valkyrie_gazebo_pkg.xacro"/>
     <xacro:include filename="$(find val_description)/model/robots/common/xacro/gazebo_harness.xacro"/>
     <xacro:include filename="$(find val_description)/model/robots/common/xacro/gazebo_self_collide.xacro"/>

File: model/robots/valkyrie_sim_arm_mass_sims.xacro (robot description, xacro)
@@ -1,3 +1,4 @@
 <robot xmlns:xacro="http://ros.org/wiki/xacro" name="valkyrie">
+    <xacro:property name="mesh_root" value="package://val_description/model/meshes"/>
     <gazebo>
       <plugin filename="libval_gazebo.so" name="SharedMemorySimInterfacePlugin">

File: model/robots/valkyrie_sim_gazebo_sync.xacro (robot description, xacro)
@@ -1,3 +1,4 @@
 <robot xmlns:xacro="http://ros.org/wiki/xacro" name="valkyrie">
+    <xacro:property name="mesh_root" value="package://val_description/model/meshes"/>
     <gazebo>
       <plugin filename="libval_gazebo.so" name="SharedMemorySimInterfacePlugin">

Commit message: adding back in double imu xacro

File: model/robots/common/xacro/pelvis/pelvis.xacro (robot description, xacro)
@@ -37,3 +37,19 @@
                                   origin_rpy="${PelvisMiddleImuFrameOrientation_RPY}" />
     </xacro:macro>
+    <xacro:macro name="v1_pelvis_sensors_usb" params="middle_sensor_node_tag middle_sensor_api_tag middle_sensor_port_tag rear_sensor_node_tag rear_sensor_api_tag rear_sensor_port_tag">
+            <xacro:usb_microstrain_sensor sensorName="pelvisRearImu"
+                                      parentLink="${Pelvis_Link_Name}"
+                                      origin_xyz="-0.075844901 0.0 -0.111056426"
+                                      origin_rpy="-3.14159 0.476467 -3.14159"
+                                      sensor_node="${rear_sensor_node_tag}"
+                                      sensor_api="${rear_sensor_api_tag}"
+                                      sensor_port="${rear_sensor_port_tag}" />
+            <xacro:usb_microstrain_sensor sensorName="pelvisMiddleImu"
+                                      parentLink="${Pelvis_Link_Name}"
+                                      origin_xyz="0.0 0.0 -0.10819638"
+                                      origin_rpy="3.14159 0.0 0.0"
+                                      sensor_node="${middle_sensor_node_tag}"
+                                      sensor_api="${middle_sensor_api_tag}"
+                                      sensor_port="${middle_sensor_port_tag}" />
+        </xacro:macro>
 </robot>

Commit message: updating imu location for testing

File: model/robots/common/xacro/pelvis/pelvis.xacro (robot description, xacro)
@@ -14,6 +14,6 @@
         <xacro:imu_sensor sensorName="pelvisRearImu"
                                   parentLink="${Pelvis_Link_Name}"
-                                  origin_xyz="-0.075844901 0.0 -0.111056426"
-                                  origin_rpy="-3.14159 0.476467 -3.14159" />
+                                  origin_xyz="0.03 0.1116 -0.1833"
+                                  origin_rpy="3.14159 0.0 0.0" />
         <xacro:imu_sensor sensorName="pelvisMiddleImu"
                                   parentLink="${Pelvis_Link_Name}"
@@ -52,6 +52,6 @@
         <xacro:usb_imu_sensor sensorName="pelvisRearImu"
                                   parentLink="${Pelvis_Link_Name}"
-                                  origin_xyz="-0.075844901 0.0 -0.111056426"
-                                  origin_rpy="-3.14159 0.476467 -3.14159"
+                                  origin_xyz="0.03 0.1116 -0.1833"
+                                  origin_rpy="3.14159 0.0 0.0"
                                   sensor_node="${rear_sensor_node_tag}"
                                   sensor_api="${rear_sensor_api_tag}"

File: model/robots/common/xacro/sensors/sensor_transforms.xacro (robot description, xacro)
@@ -1,6 +1,8 @@
 <?xml version="1.0" ?>
 <robot xmlns:xacro="http://www.ros.org/wiki/xacro" name="v1/arm/dh_parameters">
-	<xacro:property name="PelvisRearImuFrameOrigin_XYZ" value="-0.075844901 0.0 -0.111056426"/>
-	<xacro:property name="PelvisRearImuFrameOrientation_RPY" value="-3.14159 0.476467 -3.14159"/>
+	<!--<xacro:property name="PelvisRearImuFrameOrigin_XYZ" value="-0.075844901 0.0 -0.111056426"/>
+	<xacro:property name="PelvisRearImuFrameOrientation_RPY" value="-3.14159 0.476467 -3.14159"/> -->
+	<xacro:property name="PelvisRearImuFrameOrigin_XYZ" value="0.03 0.1116 -0.1833"/>
+	<xacro:property name="PelvisRearImuFrameOrientation_RPY" value="3.14159 0 0"/>
 	<xacro:property name="PelvisMiddleImuFrameOrigin_XYZ" value="0.0 0.0 -0.10819638"/>
 	<xacro:property name="PelvisMiddleImuFrameOrientation_RPY" value="3.14159 0.0 0.0"/>
