Commit message: changed mass parameters for the lighter mass sim

File: model/robots/common/xacro/waist/mass_parameters.xacro (robot description, xacro)
@@ -17,11 +17,11 @@
   <xacro:property name="TorsoPitchLinkInertia_IYZ" value="0.000000000" />
   <xacro:property name="TorsoPitchLinkInertia_IZZ" value="0.000028285" />
-  <xacro:property name="TorsoRollLinkMass" value="39.470000" />
+  <xacro:property name="TorsoRollLinkMass" value="30.870000" />
   <xacro:property name="TorsoRollLinkComPosition" value="-0.095548 -0.003337 0.243098" />
-  <xacro:property name="TorsoRollLinkInertia_IXX" value="0.87326933" />
+  <xacro:property name="TorsoRollLinkInertia_IXX" value="0.858969" />
   <xacro:property name="TorsoRollLinkInertia_IXY" value="0.000099563" />
   <xacro:property name="TorsoRollLinkInertia_IXZ" value="0.061345211" />
-  <xacro:property name="TorsoRollLinkInertia_IYY" value="1.0108485" />
+  <xacro:property name="TorsoRollLinkInertia_IYY" value="0.99655" />
   <xacro:property name="TorsoRollLinkInertia_IYZ" value="0.001818490" />
-  <xacro:property name="TorsoRollLinkInertia_IZZ" value="0.77839801" />
+  <xacro:property name="TorsoRollLinkInertia_IZZ" value="0.764098" />
 </robot>
