Commit message: updating names for remote multisense sl

File: model/urdf/multisense_sl_remote.urdf (robot description, URDF)
Before this commit: robot multisense_sl, 12 links, 11 joints
Links:
- removed link center_bottom_led_frame
- removed link center_top_led_frame
- removed link head
- removed link head_hokuyo_frame
- removed link head_imu_link
- removed link hokuyo_link
- removed link left_camera_frame
- removed link left_camera_optical_frame
- removed link left_led_frame
- removed link right_camera_frame
- removed link right_camera_optical_frame
- removed link right_led_frame
- added link multisense/center_bottom_led_frame, mass 1e-5
- added link multisense/center_top_led_frame, mass 1e-5
- added link multisense/head, mass 1.41984; collision box size=0.0468 0.12 0.1184; collision box size=0.1311 0.12 0.0591
- added link multisense/head_hokuyo_frame, mass 1e-5
- added link multisense/head_imu_link, mass 1e-5; visual box size=0.01 0.01 0.01
- added link multisense/hokuyo_link, mass 0.057654; collision box size=0.08 0.06 0.04238; collision cylinder length=0.047 radius=0.024425
- added link multisense/left_camera_frame, mass 1e-5
- added link multisense/left_camera_optical_frame
- added link multisense/left_led_frame, mass 1e-5
- added link multisense/right_camera_frame, mass 1e-5
- added link multisense/right_camera_optical_frame
- added link multisense/right_led_frame, mass 1e-5
Joints:
- joint center_bottom_led_frame_joint: child center_bottom_led_frame -> multisense/center_bottom_led_frame; parent head -> multisense/head
- joint center_top_led_frame_joint: child center_top_led_frame -> multisense/center_top_led_frame; parent head -> multisense/head
- joint head_hokuyo_joint: child head_hokuyo_frame -> multisense/head_hokuyo_frame; parent hokuyo_link -> multisense/hokuyo_link
- joint head_imu_joint: child head_imu_link -> multisense/head_imu_link; parent head -> multisense/head
- joint hokuyo_joint: child hokuyo_link -> multisense/hokuyo_link; parent head -> multisense/head
- joint left_camera_frame_joint: child left_camera_frame -> multisense/left_camera_frame; parent head -> multisense/head
- joint left_camera_optical_frame_joint: child left_camera_optical_frame -> multisense/left_camera_optical_frame; parent left_camera_frame -> multisense/left_camera_frame
- joint left_led_frame_joint: child left_led_frame -> multisense/left_led_frame; parent head -> multisense/head
- joint right_camera_frame_joint: child right_camera_frame -> multisense/right_camera_frame; parent head -> multisense/head
- joint right_camera_optical_frame_joint: child right_camera_optical_frame -> multisense/right_camera_optical_frame; parent right_camera_frame -> multisense/right_camera_frame
- joint right_led_frame_joint: child right_led_frame -> multisense/right_led_frame; parent head -> multisense/head
