Commit message: adding reflect variable for fingers for sim

File: model/robots/common/xacro/generic_models.xacro (robot description, xacro)
@@ -252,5 +252,5 @@
     </transmission>
   </xacro:macro>
-  <xacro:macro name="simple_effort_transmission_with_one_child_joint" params="jointName actuatorName nodeName actuatorApi child1JointName child1Ratio">
+  <xacro:macro name="simple_effort_transmission_with_one_child_joint" params="jointName actuatorName nodeName actuatorApi child1JointName child1Ratio reflect">
     <transmission name="${jointName}Transmission">
       <type>transmission_interface/SimpleTransmission</type>
@@ -261,10 +261,10 @@
       <actuator name="${actuatorName}">
         <node name="${nodeName}"/>
-        <mechanicalReduction>1</mechanicalReduction>
-        <api name="${actuatorApi}" />
-      </actuator>
-    </transmission>
-  </xacro:macro>
-  <xacro:macro name="simple_effort_transmission_with_three_child_joints" params="jointName actuatorName nodeName actuatorApi child1JointName child1Ratio child2JointName child2Ratio child3JointName child3Ratio">
+        <mechanicalReduction>${reflect}</mechanicalReduction>
+        <api name="${actuatorApi}" />
+      </actuator>
+    </transmission>
+  </xacro:macro>
+  <xacro:macro name="simple_effort_transmission_with_three_child_joints" params="jointName actuatorName nodeName actuatorApi child1JointName child1Ratio child2JointName child2Ratio child3JointName child3Ratio reflect">
     <transmission name="${jointName}Transmission">
       <type>transmission_interface/SimpleTransmission</type>
@@ -277,5 +277,5 @@
       <actuator name="${actuatorName}">
         <node name="${nodeName}"/>
-        <mechanicalReduction>1</mechanicalReduction>
+        <mechanicalReduction>${reflect}</mechanicalReduction>
         <api name="${actuatorApi}" />
       </actuator>

File: model/robots/common/xacro/middle_finger/middle_finger.xacro (robot description, xacro)
@@ -83,6 +83,6 @@
     <xacro:simple_forearm_position_transmission jointName="${prefix}${MiddleFingerPitch3JointName}" actuatorName="${prefix}MiddlePitch3Actuator" nodeName="/${prefix}${MiddleFingerPitch3Node}" actuatorApi="${MiddleFingerDistalApi}" reflect="${reflect}"/>
   </xacro:macro>
-  <xacro:macro name="middle_finger_transmissions_sim" params="prefix">
-    <xacro:simple_effort_transmission_with_three_child_joints jointName="${prefix}${MiddleFingerPitch1ActuatorName}" actuatorName="${prefix}${MiddleFingerPitch1ActuatorName}" nodeName="/${prefix}${MiddleFingerNode}" actuatorApi="${SimApi}" child1JointName="${prefix}${MiddleFingerPitch1JointName}" child1Ratio="${Pulley1Ratio}" child2JointName="${prefix}${MiddleFingerPitch2JointName}" child2Ratio="${Pulley2Ratio}" child3JointName="${prefix}${MiddleFingerPitch3JointName}" child3Ratio="${Pulley3Ratio}"/>
+  <xacro:macro name="middle_finger_transmissions_sim" params="prefix reflect">
+    <xacro:simple_effort_transmission_with_three_child_joints jointName="${prefix}${MiddleFingerPitch1ActuatorName}" actuatorName="${prefix}${MiddleFingerPitch1ActuatorName}" nodeName="/${prefix}${MiddleFingerNode}" actuatorApi="${SimApi}" child1JointName="${prefix}${MiddleFingerPitch1JointName}" child1Ratio="${Pulley1Ratio}" child2JointName="${prefix}${MiddleFingerPitch2JointName}" child2Ratio="${Pulley2Ratio}" child3JointName="${prefix}${MiddleFingerPitch3JointName}" child3Ratio="${Pulley3Ratio}" reflect="reflect"/>
     <xacro:simple_passive_transmission jointName="${prefix}${MiddleFingerPitch1JointName}" nodeName="/${prefix}${MiddleFingerPitch1Node}" apiName="${SimApi}" reflect="1"/>
     <xacro:simple_passive_transmission jointName="${prefix}${MiddleFingerPitch2JointName}" nodeName="/${prefix}${MiddleFingerPitch2Node}" apiName="${SimApi}" reflect="1"/>

File: model/robots/common/xacro/valkyrie_base_sim.xacro (robot description, xacro)
@@ -26,11 +26,11 @@
     <xacro:arm_transmissions_sim prefix="right"/>
     <xacro:neck_transmissions_sim />
-    <xacro:thumb_transmissions_sim prefix="left"/>
-    <xacro:thumb_transmissions_sim prefix="right"/>
-    <xacro:index_finger_transmissions_sim prefix="left"/>
-    <xacro:index_finger_transmissions_sim prefix="right"/>
-    <xacro:middle_finger_transmissions_sim prefix="left"/>
-    <xacro:middle_finger_transmissions_sim prefix="right"/>
-    <xacro:pinky_transmissions_sim prefix="left"/>
-    <xacro:pinky_transmissions_sim prefix="right"/>
+    <xacro:thumb_transmissions_sim prefix="left" reflect="-1"/>
+    <xacro:thumb_transmissions_sim prefix="right" reflect="1"/>
+    <xacro:index_finger_transmissions_sim prefix="left" reflect="-1"/>
+    <xacro:index_finger_transmissions_sim prefix="right" reflect="1"/>
+    <xacro:middle_finger_transmissions_sim prefix="left" reflect="-1"/>
+    <xacro:middle_finger_transmissions_sim prefix="right" reflect="1"/>
+    <xacro:pinky_transmissions_sim prefix="left" reflect="-1"/>
+    <xacro:pinky_transmissions_sim prefix="right" reflect="1"/>
 </robot>

Commit message: moving where reflect gets applied

File: model/robots/common/xacro/generic_models.xacro (robot description, xacro)
@@ -257,9 +257,9 @@
       <joint name="${jointName}">
         <hardwareInterface>EffortJointInterface</hardwareInterface>
-        <child name="${child1JointName}" ratio="${child1Ratio}"/>
-      </joint>
-      <actuator name="${actuatorName}">
-        <node name="${nodeName}"/>
-        <mechanicalReduction>${reflect}</mechanicalReduction>
+        <child name="${child1JointName}" ratio="${reflect}*${child1Ratio}"/>
+      </joint>
+      <actuator name="${actuatorName}">
+        <node name="${nodeName}"/>
+        <mechanicalReduction>1</mechanicalReduction>
         <api name="${actuatorApi}" />
       </actuator>
@@ -271,11 +271,11 @@
       <joint name="${jointName}">
         <hardwareInterface>EffortJointInterface</hardwareInterface>
-        <child name="${child1JointName}" ratio="${child1Ratio}"/>
-        <child name="${child2JointName}" ratio="${child2Ratio}"/>
-        <child name="${child3JointName}" ratio="${child3Ratio}"/>
-      </joint>
-      <actuator name="${actuatorName}">
-        <node name="${nodeName}"/>
-        <mechanicalReduction>${reflect}</mechanicalReduction>
+        <child name="${child1JointName}" ratio="${reflect}*${child1Ratio}"/>
+        <child name="${child2JointName}" ratio="${reflect}*${child2Ratio}"/>
+        <child name="${child3JointName}" ratio="${reflect}*${child3Ratio}"/>
+      </joint>
+      <actuator name="${actuatorName}">
+        <node name="${nodeName}"/>
+        <mechanicalReduction>1</mechanicalReduction>
         <api name="${actuatorApi}" />
       </actuator>

Commit message: correcting xacro math

File: model/robots/common/xacro/generic_models.xacro (robot description, xacro)
@@ -257,5 +257,5 @@
       <joint name="${jointName}">
         <hardwareInterface>EffortJointInterface</hardwareInterface>
-        <child name="${child1JointName}" ratio="${reflect}*${child1Ratio}"/>
+        <child name="${child1JointName}" ratio="${reflect * child1Ratio}"/>
       </joint>
       <actuator name="${actuatorName}">
@@ -271,7 +271,7 @@
       <joint name="${jointName}">
         <hardwareInterface>EffortJointInterface</hardwareInterface>
-        <child name="${child1JointName}" ratio="${reflect}*${child1Ratio}"/>
-        <child name="${child2JointName}" ratio="${reflect}*${child2Ratio}"/>
-        <child name="${child3JointName}" ratio="${reflect}*${child3Ratio}"/>
+        <child name="${child1JointName}" ratio="${reflect * child1Ratio}"/>
+        <child name="${child2JointName}" ratio="${reflect * child2Ratio}"/>
+        <child name="${child3JointName}" ratio="${reflect * child3Ratio}"/>
       </joint>
       <actuator name="${actuatorName}">
